File: hardware/edm_power_board/cad/edm_power_board/edm_power_supply.sch (KiCad schematic (older format))
At the start: 4 parts, among them U401 L78L05_SO8

Commit message: Interconnections
Other:
- moved on the sheet: U401
Changed lines of the file:
@@
 Comment4 ""
 $EndDescr
-Text HLabel 2500 2400 0    50   Input ~ 0
+Text HLabel 4400 3200 0    50   Input ~ 0
 +24V
-Text HLabel 2500 2750 0    50   Input ~ 0
+Text HLabel 4400 3550 0    50   Input ~ 0
 GNDPWR
-Text HLabel 9300 2400 2    50   Input ~ 0
+Text HLabel 7300 3200 2    50   Input ~ 0
 +5V
 $Comp
 L Regulator_Linear:L78L05_SO8 U401
 U 1 1 5A73A8F1
-P 7800 2400
-F 0 "U401" H 7800 2642 50  0000 C CNN
-F 1 "L78L05_SO8" H 7800 2551 50  0000 C CNN
-F 2 "Package_SOIC:SOIC-8_3.9x4.9mm_P1.27mm" H 7900 2600 50  0001 C CIN
-F 3 "http://www.st.com/content/ccc/resource/technical/document/datasheet/15/55/e5/aa/23/5b/43/fd/CD00000446.pdf/files/CD00000446.pdf/jcr:content/translations/en.CD00000446.pdf" H 8000 2400 50  0001 C CNN
-	1    7800 2400
+P 5800 3200
+F 0 "U401" H 5800 3442 50  0000 C CNN
+F 1 "L78L05_SO8" H 5800 3351 50  0000 C CNN
+F 2 "Package_SOIC:SOIC-8_3.9x4.9mm_P1.27mm" H 5900 3400 50  0001 C CIN
+F 3 "http://www.st.com/content/ccc/resource/technical/document/datasheet/15/55/e5/aa/23/5b/43/fd/CD00000446.pdf/files/CD00000446.pdf/jcr:content/translations/en.CD00000446.pdf" H 6000 3200 50  0001 C CNN
+	1    5800 3200
 	1    0    0    -1
 $EndComp
@@
 L Device:C C401
 U 1 1 5A73AA04
-P 7200 2650
-F 0 "C401" H 7315 2696 50  0000 L CNN
-F 1 "330n" H 7315 2605 50  0000 L CNN
-F 2 "" H 7238 2500 50  0001 C CNN
-F 3 "~" H 7200 2650 50  0001 C CNN
-	1    7200 2650
+P 5200 3450
+F 0 "C401" H 5315 3496 50  0000 L CNN
+F 1 "330n" H 5315 3405 50  0000 L CNN
+F 2 "" H 5238 3300 50  0001 C CNN
+F 3 "~" H 5200 3450 50  0001 C CNN
+	1    5200 3450
 	1    0    0    -1
 $EndComp
@@
 L Device:C C402
 U 1 1 5A73AADF
-P 8300 2650
-F 0 "C402" H 8415 2696 50  0000 L CNN
-F 1 "100n" H 8415 2605 50  0000 L CNN
-F 2 "" H 8338 2500 50  0001 C CNN
-F 3 "~" H 8300 2650 50  0001 C CNN
-	1    8300 2650
+P 6300 3450
+F 0 "C402" H 6415 3496 50  0000 L CNN
+F 1 "100n" H 6415 3405 50  0000 L CNN
+F 2 "" H 6338 3300 50  0001 C CNN
+F 3 "~" H 6300 3450 50  0001 C CNN
+	1    6300 3450
 	1    0    0    -1
 $EndComp
@@
 L power:GNDPWR #PWR030
 U 1 1 5A73AD03
-P 7200 3100
-F 0 "#PWR030" H 7200 2900 50  0001 C CNN
-F 1 "GNDPWR" H 7200 2900 50  0000 C CNN
-F 2 "" H 7200 3050 50  0001 C CNN
-F 3 "" H 7200 3050 50  0001 C CNN
-	1    7200 3100
+P 5200 3900
+F 0 "#PWR030" H 5200 3700 50  0001 C CNN
+F 1 "GNDPWR" H 5200 3700 50  0000 C CNN
+F 2 "" H 5200 3850 50  0001 C CNN
+F 3 "" H 5200 3850 50  0001 C CNN
+	1    5200 3900
 	1    0    0    -1
 $EndComp
@@
 L power:GNDPWR #PWR031
 U 1 1 5A73AD3E
-P 2700 2950
-F 0 "#PWR031" H 2700 2750 50  0001 C CNN
-F 1 "GNDPWR" H 2700 2750 50  0000 C CNN
-F 2 "" H 2700 2900 50  0001 C CNN
-F 3 "" H 2700 2900 50  0001 C CNN
-	1    2700 2950
+P 4600 3750
+F 0 "#PWR031" H 4600 3550 50  0001 C CNN
+F 1 "GNDPWR" H 4600 3550 50  0000 C CNN
+F 2 "" H 4600 3700 50  0001 C CNN
+F 3 "" H 4600 3700 50  0001 C CNN
+	1    4600 3750
 	1    0    0    -1
 $EndComp
 Wire Wire Line
-	2500 2400 7200 2400
+	6100 3200 6300 3200
 Wire Wire Line
-	8100 2400 8300 2400
+	6300 3300 6300 3200
+Connection ~ 6300 3200
 Wire Wire Line
-	8300 2500 8300 2400
-Connection ~ 8300 2400
+	6300 3200 6750 3200
 Wire Wire Line
-	8300 2400 8750 2400
+	5200 3300 5200 3200
 Wire Wire Line
-	7200 2500 7200 2400
-Connection ~ 7200 2400
+	5200 3200 5500 3200
 Wire Wire Line
-	7200 2400 7500 2400
+	4400 3550 4600 3550
 Wire Wire Line
-	2500 2750 2700 2750
+	4600 3550 4600 3750
 Wire Wire Line
-	2700 2750 2700 2950
+	5200 3900 5200 3700
 Wire Wire Line
-	7200 3100 7200 2900
+	5200 3700 5800 3700
 Wire Wire Line
-	7200 2900 7800 2900
+	5800 3700 5800 3500
+Connection ~ 5200 3700
 Wire Wire Line
-	7800 2900 7800 2700
-Connection ~ 7200 2900
+	5200 3700 5200 3600
 Wire Wire Line
-	7200 2900 7200 2800
+	5800 3700 6300 3700
 Wire Wire Line
-	7800 2900 8300 2900
-Wire Wire Line
-	8300 2900 8300 2800
-Connection ~ 7800 2900
+	6300 3700 6300 3600
+Connection ~ 5800 3700
 $Comp
 L Device:C C403
 U 1 1 5A73B168
-P 8750 2650
-F 0 "C403" H 8865 2696 50  0000 L CNN
-F 1 "1u" H 8865 2605 50  0000 L CNN
-F 2 "" H 8788 2500 50  0001 C CNN
-F 3 "~" H 8750 2650 50  0001 C CNN
-	1    8750 2650
+P 6750 3450
+F 0 "C403" H 6865 3496 50  0000 L CNN
+F 1 "1u" H 6865 3405 50  0000 L CNN
+F 2 "" H 6788 3300 50  0001 C CNN
+F 3 "~" H 6750 3450 50  0001 C CNN
+	1    6750 3450
 	1    0    0    -1
 $EndComp
 Wire Wire Line
-	8750 2500 8750 2400
-Connection ~ 8750 2400
+	6750 3300 6750 3200
+Connection ~ 6750 3200
 Wire Wire Line
-	8750 2400 9300 2400
+	6750 3200 7300 3200
 Wire Wire Line
-	8300 2900 8750 2900
+	6300 3700 6750 3700
 Wire Wire Line
-	8750 2900 8750 2800
-Connection ~ 8300 2900
+	6750 3700 6750 3600
+Connection ~ 6300 3700
+Wire Wire Line
+	4400 3200 5200 3200
+Connection ~ 5200 3200
 $EndSCHEMATC

Commit message: Assign part numbers
Parts:
- C401: footprint (none) -> Capacitor_SMD:C_0805_2012Metric; Digikey (none) -> 1276-6813-1-ND
- C402: footprint (none) -> Capacitor_SMD:C_0805_2012Metric; Digikey (none) -> 445-1418-1-ND
- C403: footprint (none) -> Capacitor_SMD:C_0805_2012Metric; Digikey (none) -> 1276-1066-1-ND
- U401: Digikey (none) -> 497-1182-1-ND
Changed lines of the file:
@@
 F 2 "Package_SOIC:SOIC-8_3.9x4.9mm_P1.27mm" H 5900 3400 50  0001 C CIN
 F 3 "http://www.st.com/content/ccc/resource/technical/document/datasheet/15/55/e5/aa/23/5b/43/fd/CD00000446.pdf/files/CD00000446.pdf/jcr:content/translations/en.CD00000446.pdf" H 6000 3200 50  0001 C CNN
+F 4 "497-1182-1-ND" H 5800 3200 50  0001 C CNN "Digikey"
 	1    5800 3200
 	1    0    0    -1
@@
 F 0 "C401" H 5315 3496 50  0000 L CNN
 F 1 "330n" H 5315 3405 50  0000 L CNN
-F 2 "" H 5238 3300 50  0001 C CNN
+F 2 "Capacitor_SMD:C_0805_2012Metric" H 5238 3300 50  0001 C CNN
 F 3 "~" H 5200 3450 50  0001 C CNN
+F 4 "1276-6813-1-ND" H 5200 3450 50  0001 C CNN "Digikey"
 	1    5200 3450
 	1    0    0    -1
@@
 F 0 "C402" H 6415 3496 50  0000 L CNN
 F 1 "100n" H 6415 3405 50  0000 L CNN
-F 2 "" H 6338 3300 50  0001 C CNN
+F 2 "Capacitor_SMD:C_0805_2012Metric" H 6338 3300 50  0001 C CNN
 F 3 "~" H 6300 3450 50  0001 C CNN
+F 4 "445-1418-1-ND" H 6300 3450 50  0001 C CNN "Digikey"
 	1    6300 3450
 	1    0    0    -1
@@
 F 0 "C403" H 6865 3496 50  0000 L CNN
 F 1 "1u" H 6865 3405 50  0000 L CNN
-F 2 "" H 6788 3300 50  0001 C CNN
+F 2 "Capacitor_SMD:C_0805_2012Metric" H 6788 3300 50  0001 C CNN
 F 3 "~" H 6750 3450 50  0001 C CNN
+F 4 "1276-1066-1-ND" H 6750 3450 50  0001 C CNN "Digikey"
 	1    6750 3450
 	1    0    0    -1

Commit message: PCB Outline
Parts:
- U401: footprint Package_SOIC:SOIC-8_3.9x4.9mm_P1.27mm -> Package_SO:SOIC-8_3.9x4.9mm_P1.27mm
Changed lines of the file:
@@
 F 0 "U401" H 5800 3442 50  0000 C CNN
 F 1 "L78L05_SO8" H 5800 3351 50  0000 C CNN
-F 2 "Package_SOIC:SOIC-8_3.9x4.9mm_P1.27mm" H 5900 3400 50  0001 C CIN
+F 2 "Package_SO:SOIC-8_3.9x4.9mm_P1.27mm" H 5900 3400 50  0001 C CIN
 F 3 "http://www.st.com/content/ccc/resource/technical/document/datasheet/15/55/e5/aa/23/5b/43/fd/CD00000446.pdf/files/CD00000446.pdf/jcr:content/translations/en.CD00000446.pdf" H 6000 3200 50  0001 C CNN
 F 4 "497-1182-1-ND" H 5800 3200 50  0001 C CNN "Digikey"

Commit message: Add input capacitors to spark
Parts:
- C403: Digikey 1276-1066-1-ND -> 587-2910-1-ND
Changed lines of the file:
@@
 F 2 "Capacitor_SMD:C_0805_2012Metric" H 6788 3300 50  0001 C CNN
 F 3 "~" H 6750 3450 50  0001 C CNN
-F 4 "1276-1066-1-ND" H 6750 3450 50  0001 C CNN "Digikey"
+F 4 "587-2910-1-ND" H 6750 3450 50  0001 C CNN "Digikey"
 	1    6750 3450
 	1    0    0    -1
