File: hardware/edm_power_board/cad/edm_power_board/edm_spark_voltage_source.sch (KiCad schematic (older format))
At the start: 24 parts

Commit message: Spark voltage source
Parts:
- removed R?: 85k, symbol Device:R
- removed R?: 265R, symbol Device:R
- added C301, C303: 100n, symbol Device:C
- added C308, C309: 1u, symbol Device:C
- added C310, C311: 56u, symbol Device:CP
- added D301: 5V1, symbol Device:D_Zener
- added R303, R307: 84k5, symbol Device:R
- added R304: 21k, Resistor_SMD:R_0805_2012Metric, symbol Device:R
- added R306: 27k, Resistor_SMD:R_0805_2012Metric, symbol Device:R
- added R310, R311: 93k1, Resistor_SMD:R_1206_3216Metric, symbol Device:R
- added R312: 10k, Resistor_SMD:R_0805_2012Metric, symbol Device:R
- added R316: 261R, Resistor_SMD:R_0805_2012Metric, symbol Device:R
- added U302: Si8641xx-x-xS1, Package_SO:SOIC-16_3.9x9.9mm_P1.27mm, symbol Isolator:Si8641xx-x-xS1
- added U304: LM311, symbol Comparator:LM311
- R301: renamed from R?; footprint (none) -> Resistor_SMD:R_0805_2012Metric; DigiKey (none) -> 311-27KARCT-ND
- R302: renamed from R?; footprint (none) -> Resistor_SMD:R_0805_2012Metric; DigiKey (none) -> 311-2.20KCRCT-ND
- R305: renamed from R?; footprint (none) -> Resistor_SMD:R_0805_2012Metric; DigiKey (none) -> 311-3.00KCRCT-ND
- R308: renamed from R?; value 263R -> 261R; footprint (none) -> Resistor_SMD:R_0805_2012Metric; DigiKey (none) -> 311-261CRCT-ND
- R309: renamed from R?; value 10k55 -> 10k5; footprint (none) -> Resistor_SMD:R_0805_2012Metric; DigiKey (none) -> 311-10.5KCRCT-ND
- R313: renamed from R?; footprint (none) -> Resistor_SMD:R_0805_2012Metric; DigiKey (none) -> 311-523CRCT-ND
- R314: renamed from R?; footprint (none) -> Resistor_SMD:R_0805_2012Metric; DigiKey (none) -> 311-102CRCT-ND
- R315: renamed from R?; value 3k -> 150m; footprint (none) -> Resistor_SMD:R_1206_3216Metric; DigiKey (none) -> 311-.15LYCT-ND
- R317: renamed from R?; footprint (none) -> Resistor_SMD:R_0805_2012Metric; DigiKey (none) -> 311-21.0KCRCT-ND
- R318: renamed from R?; footprint (none) -> Resistor_SMD:R_0805_2012Metric; DigiKey (none) -> 541-180CCT-ND
- gave numbers to parts that had none: 12
Connections:
- net labels added: +24V, +250V, +3.3V, +3V3, +5V, GND
- wire segments 83 -> 175
Other:
- note added: "3.8V"

Commit message: Insulator
Parts:
- removed U302: Si8641xx-x-xS1, Package_SO:SOIC-16_3.9x9.9mm_P1.27mm, symbol Isolator:Si8641xx-x-xS1
- added U?: Si8641BB-B-IS1, Package_SO:SOIC-16_3.9x9.9mm_P1.27mm, symbol Isolator:Si8641BB-B-IS1
Connections:
- net labels added: Spark_Voltage_0, Spark_Voltage_1, Spark_Voltage_2, Spark_Voltage_Status
- wire segments 175 -> 179

Commit message: Spark output
Parts:
- added C?: 100n, symbol Device:C
Connections:
- wire segments 179 -> 181
Changed lines of the file:
@@
 Wire Wire Line
 	1700 4200 2050 4200
+$Comp
+L Device:C C?
+U 1 1 5A7D76CF
+P 4100 7100
+F 0 "C?" H 4215 7146 50  0000 L CNN
+F 1 "100n" H 4215 7055 50  0000 L CNN
+F 2 "" H 4138 6950 50  0001 C CNN
+F 3 "~" H 4100 7100 50  0001 C CNN
+	1    4100 7100
+	1    0    0    -1
+$EndComp
+$Comp
+L power:+5V #PWR?
+U 1 1 5A7D778B
+P 4100 6850
+F 0 "#PWR?" H 4100 6700 50  0001 C CNN
+F 1 "+5V" H 4115 7023 50  0000 C CNN
+F 2 "" H 4100 6850 50  0001 C CNN
+F 3 "" H 4100 6850 50  0001 C CNN
+	1    4100 6850
+	1    0    0    -1
+$EndComp
+$Comp
+L power:GNDPWR #PWR?
+U 1 1 5A7D780E
+P 4100 7350
+F 0 "#PWR?" H 4100 7150 50  0001 C CNN
+F 1 "GNDPWR" H 4100 7150 50  0000 C CNN
+F 2 "" H 4100 7300 50  0001 C CNN
+F 3 "" H 4100 7300 50  0001 C CNN
+	1    4100 7350
+	1    0    0    -1
+$EndComp
+Wire Wire Line
+	4100 7350 4100 7250
+Wire Wire Line
+	4100 6950 4100 6850
 $EndSCHEMATC

Commit message: Assign part numbers
Parts:
- removed C309: 1u, symbol Device:C
- removed C310, C311: 56u, symbol Device:CP
- removed Q303, Q304: BSS214NW, Package_TO_SOT_SMD:SOT-323_SC-70, symbol Transistor_FET:BSS214NW
- added C? (x2): 470n, Capacitor_SMD:C_1812_4532Metric, symbol Device:C
- added C? (x2): 25u, Capacitor_THT:C_Rect_L41.5mm_W20.0mm_P37.50mm_MKS4, symbol Device:C
- added Q? (x2): BSS214NW, Package_TO_SOT_SMD:SOT-323_SC-70, symbol Transistor_FET:BSS214NW
- C301, C303, C304, C?: footprint (none) -> Capacitor_SMD:C_0805_2012Metric; Digikey (none) -> 1276-1066-1-ND
- C302: footprint (none) -> Capacitor_SMD:C_0805_2012Metric; Digikey (none) -> 490-1664-1-ND
- C305: value 125n -> 120n; footprint (none) -> Capacitor_SMD:C_0805_2012Metric; Digikey (none) -> 1276-6518-1-ND
- C306: value 530p -> 560p; footprint (none) -> Capacitor_SMD:C_0805_2012Metric; Digikey (none) -> 399-3492-1-ND
- C307: footprint (none) -> Capacitor_SMD:C_0805_2012Metric; Digikey (none) -> 399-1147-1-ND
- C308: value 1u -> 470n; footprint (none) -> Capacitor_SMD:C_1812_4532Metric; Digikey (none) -> 445-13461-2-ND
- D301: value 5V1 -> 4V7; footprint (none) -> Diode_SMD:D_SOD-123; Digikey (none) -> BZT52C4V7-13FDICT-ND; Mfg part (none) -> BZT52C4V7-13-F
- D302: Digikey (none) -> 1655-1739-1-ND
- Q301: Digikey (none) -> BSS214NWH6327XTSA1CT-ND
- Q302: Digikey (none) -> BSC13DN30NSFDATMA1CT-ND
- R301, R306: DigiKey 311-27KARCT-ND -> 311-27.0KCRCT-ND
- R303: footprint (none) -> Resistor_SMD:R_0805_2012Metric
- R310, R311: DigiKey 311-93.1KFRCT-ND -> 311-93.1KCRCT-ND
- R315: footprint Resistor_SMD:R_1206_3216Metric -> Resistor_SMD:R_2512_6332Metric; DigiKey 311-.15LYCT-ND -> 311-0.15TCT-ND
- R318: DigiKey 541-180CCT-ND -> 311-180CRCT-ND
- U303: Digikey (none) -> LM5022MM/NOPBCT-ND
- U304: footprint (none) -> Package_SO:SOIC-8_3.9x4.9mm_P1.27mm; Digikey (none) -> LM311MX/NOPBCT-ND
- U?: Digikey (none) -> 336-2566-ND

Commit message: Set component references
Parts:
- gave numbers to parts that had none: 8
Changed lines of the file:
@@
 $EndComp
 $Comp
-L Isolator:Si8641BB-B-IS1 U?
+L Isolator:Si8641BB-B-IS1 U302
 U 1 1 5A79F1F6
 P 3250 5250
-F 0 "U?" H 3250 5917 50  0000 C CNN
+F 0 "U302" H 3250 5917 50  0000 C CNN
 F 1 "Si8641BB-B-IS1" H 3250 5826 50  0000 C CNN
 F 2 "Package_SO:SOIC-16_3.9x9.9mm_P1.27mm" H 3250 4700 50  0001 C CIN
@@
 Connection ~ 4200 6500
 $Comp
-L power:GNDPWR #PWR?
+L power:GNDPWR #PWR032
 U 1 1 5A841EA0
 P 3750 5750
-F 0 "#PWR?" H 3750 5550 50  0001 C CNN
+F 0 "#PWR032" H 3750 5550 50  0001 C CNN
 F 1 "GNDPWR" H 3750 5550 50  0000 C CNN
 F 2 "" H 3750 5700 50  0001 C CNN
@@
 Connection ~ 2750 4850
 $Comp
-L power:GND #PWR?
+L power:GND #PWR033
 U 1 1 5A86C02C
 P 2750 5750
-F 0 "#PWR?" H 2750 5500 50  0001 C CNN
+F 0 "#PWR033" H 2750 5500 50  0001 C CNN
 F 1 "GND" H 2755 5577 50  0000 C CNN
 F 2 "" H 2750 5750 50  0001 C CNN
@@
 	1500 4050 1850 4050
 $Comp
-L Device:C C?
+L Device:C C309
 U 1 1 5A7D76CF
 P 3650 6900
-F 0 "C?" H 3765 6946 50  0000 L CNN
+F 0 "C309" H 3765 6946 50  0000 L CNN
 F 1 "100n" H 3765 6855 50  0000 L CNN
 F 2 "Capacitor_SMD:C_0805_2012Metric" H 3688 6750 50  0001 C CNN
@@
 $EndComp
 $Comp
-L power:+5V #PWR?
+L power:+5V #PWR034
 U 1 1 5A7D778B
 P 3650 6650
-F 0 "#PWR?" H 3650 6500 50  0001 C CNN
+F 0 "#PWR034" H 3650 6500 50  0001 C CNN
 F 1 "+5V" H 3665 6823 50  0000 C CNN
 F 2 "" H 3650 6650 50  0001 C CNN
@@
 $EndComp
 $Comp
-L power:GNDPWR #PWR?
+L power:GNDPWR #PWR035
 U 1 1 5A7D780E
 P 3650 7150
-F 0 "#PWR?" H 3650 6950 50  0001 C CNN
+F 0 "#PWR035" H 3650 6950 50  0001 C CNN
 F 1 "GNDPWR" H 3650 6950 50  0000 C CNN
 F 2 "" H 3650 7100 50  0001 C CNN
@@
 	3650 6750 3650 6650
 $Comp
-L Device:C C?
+L Device:C C310
 U 1 1 5A834325
 P 8700 1550
-F 0 "C?" H 8815 1596 50  0000 L CNN
+F 0 "C310" H 8815 1596 50  0000 L CNN
 F 1 "470n" H 8815 1505 50  0000 L CNN
 F 2 "Capacitor_SMD:C_1812_4532Metric" H 8738 1400 50  0001 C CNN
@@
 Connection ~ 8700 1800
 $Comp
-L Device:C C?
+L Device:C C313
 U 1 1 5A8E5143
 P 19450 950
-F 0 "C?" H 19565 996 50  0000 L CNN
+F 0 "C313" H 19565 996 50  0000 L CNN
 F 1 "470n" H 19565 905 50  0000 L CNN
 F 2 "Capacitor_SMD:C_1812_4532Metric" H 19488 800 50  0001 C CNN
@@
 $EndComp
 $Comp
-L Device:C C?
+L Device:C C311
 U 1 1 5A8E5211
 P 9200 1550
-F 0 "C?" H 9315 1596 50  0000 L CNN
+F 0 "C311" H 9315 1596 50  0000 L CNN
 F 1 "25u" H 9315 1505 50  0000 L CNN
 F 2 "Capacitor_THT:C_Rect_L41.5mm_W20.0mm_P37.50mm_MKS4" H 9238 1400 50  0001 C CNN
@@
 $EndComp
 $Comp
-L Device:C C?
+L Device:C C312
 U 1 1 5A8EE597
 P 9750 1550
-F 0 "C?" H 9865 1596 50  0000 L CNN
+F 0 "C312" H 9865 1596 50  0000 L CNN
 F 1 "25u" H 9865 1505 50  0000 L CNN
 F 2 "Capacitor_THT:C_Rect_L41.5mm_W20.0mm_P37.50mm_MKS4" H 9788 1400 50  0001 C CNN
@@
 $EndComp
 $Comp
-L Transistor_FET:BSS214NW Q?
+L Transistor_FET:BSS214NW Q303
 U 1 1 5A8EEB3B
 P 7400 4550
-F 0 "Q?" H 7605 4596 50  0000 L CNN
+F 0 "Q303" H 7605 4596 50  0000 L CNN
 F 1 "BSS214NW" H 7605 4505 50  0000 L CNN
 F 2 "Package_TO_SOT_SMD:SOT-323_SC-70" H 7600 4475 50  0001 L CIN
@@
 $EndComp
 $Comp
-L Transistor_FET:BSS214NW Q?
+L Transistor_FET:BSS214NW Q304
 U 1 1 5A8EEBB1
 P 8400 4550
-F 0 "Q?" H 8605 4596 50  0000 L CNN
+F 0 "Q304" H 8605 4596 50  0000 L CNN
 F 1 "BSS214NW" H 8605 4505 50  0000 L CNN
 F 2 "Package_TO_SOT_SMD:SOT-323_SC-70" H 8600 4475 50  0001 L CIN

Commit message: Set part numbers
Parts:
- removed C313: 470n, Capacitor_SMD:C_1812_4532Metric, symbol Device:C
- C309: renamed from C308; Digikey 445-13461-2-ND -> 445-13461-1-ND
- C310: Digikey 445-13461-2-ND -> 445-13461-1-ND
- L301: footprint (none) -> Inductor_SMD:L_12x12mm_H8mm; Digikey (none) -> 553-3686-1-ND
- R301, R306: DigiKey 311-27.0KCRCT-ND -> (none); Digikey (none) -> 311-27.0KCRCT-ND
- R302: DigiKey 311-2.20KCRCT-ND -> (none); Digikey (none) -> 311-2.20KCRCT-ND
- R303, R307: DigiKey 311-84.5KCRCT-ND -> (none); Digikey (none) -> 311-84.5KCRCT-ND
- R304, R317: DigiKey 311-21.0KCRCT-ND -> (none); Digikey (none) -> 311-21.0KCRCT-ND
- R305: DigiKey 311-3.00KCRCT-ND -> (none); Digikey (none) -> 311-3.00KCRCT-ND
- R308, R316: DigiKey 311-261CRCT-ND -> (none); Digikey (none) -> 311-261CRCT-ND
- R309: DigiKey 311-10.5KCRCT-ND -> (none); Digikey (none) -> 311-10.5KCRCT-ND
- R310, R311: DigiKey 311-93.1KCRCT-ND -> (none); Digikey (none) -> 311-93.1KCRCT-ND
- R312: DigiKey 311-10.0KCRCT-ND -> (none); Digikey (none) -> 311-10.0KCRCT-ND
- R313: DigiKey 311-523CRCT-ND -> (none); Digikey (none) -> 311-523CRCT-ND
- R314: DigiKey 311-102CRCT-ND -> (none); Digikey (none) -> 311-102CRCT-ND
- R315: DigiKey 311-0.15TCT-ND -> (none); Digikey (none) -> 311-0.15TCT-ND
- R318: DigiKey 311-180CRCT-ND -> (none); Digikey (none) -> 311-180CRCT-ND
- renumbered C309 to C303, C303 to C304, C304 to C305, C305 to C306, C306 to C307, C307 to C308, U302 to U301, U303 to U302, U304 to U303

Commit message: PCB Outline
Parts:
- R307: footprint (none) -> Resistor_SMD:R_0805_2012Metric
- U302: footprint Package_SSOP:MSOP-10_3x3mm_P0.5mm -> Package_SO:MSOP-10_3x3mm_P0.5mm
Changed lines of the file:
@@
 F 0 "U302" H 4000 2667 50  0000 C CNN
 F 1 "LM5022MM" H 4000 2576 50  0000 C CNN
-F 2 "Package_SSOP:MSOP-10_3x3mm_P0.5mm" H 4050 1650 50  0001 L CIN
+F 2 "Package_SO:MSOP-10_3x3mm_P0.5mm" H 4050 1650 50  0001 L CIN
 F 3 "http://www.ti.com/lit/ds/symlink/lm5022.pdf" H 4000 2100 50  0001 C CNN
 F 4 "LM5022MM/NOPBCT-ND" H 4000 2100 50  0001 C CNN "Digikey"
@@
 F 0 "R307" H 5270 6896 50  0000 L CNN
 F 1 "84k5" H 5270 6805 50  0000 L CNN
-F 2 "" V 5130 6850 50  0001 C CNN
+F 2 "Resistor_SMD:R_0805_2012Metric" V 5130 6850 50  0001 C CNN
 F 3 "~" H 5200 6850 50  0001 C CNN
 F 4 "311-84.5KCRCT-ND" H 5200 6850 50  0001 C CNN "Digikey"

Commit message: Add input capacitors to spark
Parts:
- added C301: CP, symbol Device:CP
- added C302, C304, C305: 1u, Capacitor_SMD:C_0805_2012Metric, symbol Device:C
- C309: renamed from C305; Digikey 1276-1066-1-ND -> 587-2910-1-ND
- renumbered C301 to C303, C302 to C306, C303 to C307, C304 to C308, C306 to C310, C307 to C311, C308 to C312, C309 to C313, C310 to C314, C311 to C315, C312 to C316
Connections:
- wire segments 181 -> 198
