File: hardware/edm_power_board/cad/edm_power_board/edm_spark_voltage_source.sch (KiCad schematic (older format))
At the start: 44 parts, among them Q301 BSS214NW, Q302 BSC13DN30NSFD, Q303 BSS214NW, Q304 BSS214NW, U301 Si8641BB-B-IS1, U302 LM5022MM, U303 LM311

Commit message: Component placement 250V
Parts:
- C301: value CP -> 22u; footprint (none) -> Capacitor_SMD:CP_Elec_5x5.3; Digikey (none) -> PCE4240CT-ND
Changed lines of the file:
@@
 P 1750 1350
 F 0 "C301" H 1868 1396 50  0000 L CNN
-F 1 "CP" H 1868 1305 50  0000 L CNN
-F 2 "" H 1788 1200 50  0001 C CNN
+F 1 "22u" H 1868 1305 50  0000 L CNN
+F 2 "Capacitor_SMD:CP_Elec_5x5.3" H 1788 1200 50  0001 C CNN
 F 3 "~" H 1750 1350 50  0001 C CNN
+F 4 "PCE4240CT-ND" H 1750 1350 50  0001 C CNN "Digikey"
 	1    1750 1350
 	1    0    0    -1

Commit message: Plated mounting holes
Parts:
- U301: value Si8641BB-B-IS1 -> Si8641BB-B-IS; footprint Package_SO:SOIC-16_3.9x9.9mm_P1.27mm -> Package_SO:SOIC-16W_7.5x10.3mm_P1.27mm; symbol Isolator:Si8641BB-B-IS1 -> Isolator:Si8641BB-B-IS; Digikey 336-2566-ND -> SI8641BB-B-IS-ND
Changed lines of the file:
@@
 $EndComp
 $Comp
-L Isolator:Si8641BB-B-IS1 U301
+L Isolator:Si8641BB-B-IS U301
 U 1 1 5A79F1F6
 P 3250 5250
 F 0 "U301" H 3250 5917 50  0000 C CNN
-F 1 "Si8641BB-B-IS1" H 3250 5826 50  0000 C CNN
-F 2 "Package_SO:SOIC-16_3.9x9.9mm_P1.27mm" H 3250 4700 50  0001 C CIN
+F 1 "Si8641BB-B-IS" H 3250 5826 50  0000 C CNN
+F 2 "Package_SO:SOIC-16W_7.5x10.3mm_P1.27mm" H 3250 4700 50  0001 C CIN
 F 3 "https://www.silabs.com/documents/public/data-sheets/si864x-datasheet.pdf" H 3250 5650 50  0001 C CNN
-F 4 "336-2566-ND" H 3250 5250 50  0001 C CNN "Digikey"
+F 4 "SI8641BB-B-IS-ND" H 3250 5250 50  0001 C CNN "Digikey"
 	1    3250 5250
 	1    0    0    -1

Commit message: Component placement
Parts:
- L301: footprint Inductor_SMD:L_12x12mm_H8mm -> Inductor_SMD:L_Pulse_PA4320
Changed lines of the file:
@@
 F 0 "L301" V 5590 1300 50  0000 C CNN
 F 1 "1m" V 5499 1300 50  0000 C CNN
-F 2 "Inductor_SMD:L_12x12mm_H8mm" H 5400 1300 50  0001 C CNN
+F 2 "Inductor_SMD:L_Pulse_PA4320" H 5400 1300 50  0001 C CNN
 F 3 "http://productfinder.pulseeng.com/products/datasheets/P787.pdf" H 5400 1300 50  0001 C CNN
 F 4 "553-3686-1-ND" V 5400 1300 50  0001 C CNN "Digikey"

Commit message: Routing
Connections:
- net labels added: VS_COMP, VS_CS, VS_CS2, VS_FB, VS_OUT, VS_QD, VS_QS, VS_RT, VS_UVLO, VS_VCC, VS_VIN
Changed lines of the file:
@@
 Wire Wire Line
 	3500 1050 3500 1300
+Text Label 4450 1800 0    50   ~ 0
+VS_OUT
+Text Label 4450 1900 0    50   ~ 0
+VS_CS
+Text Label 4450 2100 0    50   ~ 0
+VS_FB
+Text Label 4450 2200 0    50   ~ 0
+VS_COMP
+Text Label 4450 2400 0    50   ~ 0
+VS_VCC
+Text Label 3200 2200 0    50   ~ 0
+VS_RT
+Text Label 3200 2000 0    50   ~ 0
+VS_UVLO
+Text Label 3200 1800 0    50   ~ 0
+VS_VIN
+Text Label 6300 2500 1    50   ~ 0
+VS_CS2
+Text Label 6800 2450 1    50   ~ 0
+VS_QS
+Text Label 6800 1550 1    50   ~ 0
+VS_QD
 $EndSCHEMATC
