File: hardware/edm_power_board/cad/edm_power_board/edm_connectors.sch (KiCad schematic (older format))
At the start: 0 parts

Commit message: Interconnections
Parts:
- added J?: Conn_02x08_Odd_Even, symbol Connector_Generic:Conn_02x08_Odd_Even
- added J?: Conn_01x02, symbol Connector_Generic:Conn_01x02
Connections:
- net labels added: +3V3, Breakdown, GND, Output_20V_Enable, Output_250V_Enable, Short_Circuit, Spark_Voltage_0, Spark_Voltage_1, Spark_Voltage_2, Spark_Voltage_Status
- wire segments 0 -> 25
Changed lines of the file:
@@
 Comment4 ""
 $EndDescr
-Text HLabel 9400 2400 2    50   Input ~ 0
+Text HLabel 5100 4000 0    50   Input ~ 0
 +24V
-Text HLabel 9400 2800 2    50   Input ~ 0
+Text HLabel 5100 4100 0    50   Input ~ 0
 GNDPWR
+$Comp
+L Connector_Generic:Conn_02x08_Odd_Even J?
+U 1 1 5A7A474C
+P 5600 2800
+F 0 "J?" H 5650 3317 50  0000 C CNN
+F 1 "Conn_02x08_Odd_Even" H 5650 3226 50  0000 C CNN
+F 2 "" H 5600 2800 50  0001 C CNN
+F 3 "~" H 5600 2800 50  0001 C CNN
+	1    5600 2800
+	1    0    0    -1
+$EndComp
+Text HLabel 6400 2500 2    50   Input ~ 0
+Output_250V_Enable
+Text HLabel 6400 2600 2    50   Input ~ 0
+Output_20V_Enable
+Text HLabel 6400 2700 2    50   Input ~ 0
+Short_Circuit
+Text HLabel 6400 2800 2    50   Input ~ 0
+Breakdown
+Text HLabel 6400 2900 2    50   Input ~ 0
+Spark_Voltage_0
+Text HLabel 6400 3000 2    50   Input ~ 0
+Spark_Voltage_1
+Text HLabel 6400 3100 2    50   Input ~ 0
+Spark_Voltage_2
+Text HLabel 6400 3200 2    50   Input ~ 0
+Spark_Voltage_Status
+Text HLabel 5100 2500 0    50   Input ~ 0
++3V3
+Text HLabel 5100 2600 0    50   Input ~ 0
+GND
+Wire Wire Line
+	5100 2600 5300 2600
+Wire Wire Line
+	5300 2600 5300 2700
+Wire Wire Line
+	5300 3200 5400 3200
+Connection ~ 5300 2600
+Wire Wire Line
+	5300 2600 5400 2600
+Wire Wire Line
+	5400 3100 5300 3100
+Connection ~ 5300 3100
+Wire Wire Line
+	5300 3100 5300 3200
+Wire Wire Line
+	5300 3000 5400 3000
+Connection ~ 5300 3000
+Wire Wire Line
+	5300 3000 5300 3100
+Wire Wire Line
+	5400 2900 5300 2900
+Connection ~ 5300 2900
+Wire Wire Line
+	5300 2900 5300 3000
+Wire Wire Line
+	5300 2800 5400 2800
+Connection ~ 5300 2800
+Wire Wire Line
+	5300 2800 5300 2900
+Wire Wire Line
+	5400 2700 5300 2700
+Connection ~ 5300 2700
+Wire Wire Line
+	5300 2700 5300 2800
+Wire Wire Line
+	5100 2500 5400 2500
+Wire Wire Line
+	5900 2500 6400 2500
+Wire Wire Line
+	6400 2600 5900 2600
+Wire Wire Line
+	5900 2700 6400 2700
+Wire Wire Line
+	6400 2800 5900 2800
+Wire Wire Line
+	5900 2900 6400 2900
+Wire Wire Line
+	6400 3000 5900 3000
+Wire Wire Line
+	5900 3100 6400 3100
+Wire Wire Line
+	6400 3200 5900 3200
+$Comp
+L Connector_Generic:Conn_01x02 J?
+U 1 1 5A7F6FB6
+P 5600 4000
+F 0 "J?" H 5680 3992 50  0000 L CNN
+F 1 "Conn_01x02" H 5680 3901 50  0000 L CNN
+F 2 "" H 5600 4000 50  0001 C CNN
+F 3 "~" H 5600 4000 50  0001 C CNN
+	1    5600 4000
+	1    0    0    -1
+$EndComp
+Wire Wire Line
+	5100 4000 5400 4000
+Wire Wire Line
+	5400 4100 5100 4100
 $EndSCHEMATC

Commit message: Assign part numbers
Parts:
- J?: footprint (none) -> Connector_PinHeader_1.27mm:PinHeader_2x08_P1.27mm_Vertical; Digikey (none) -> ED10523-ND
- J?: footprint (none) -> TerminalBlock:TerminalBlock_bornier-2_P5.08mm; Digikey (none) -> ED1609-ND
Changed lines of the file:
@@
 F 0 "J?" H 5650 3317 50  0000 C CNN
 F 1 "Conn_02x08_Odd_Even" H 5650 3226 50  0000 C CNN
-F 2 "" H 5600 2800 50  0001 C CNN
-F 3 "~" H 5600 2800 50  0001 C CNN
+F 2 "Connector_PinHeader_1.27mm:PinHeader_2x08_P1.27mm_Vertical" H 5600 2800 50  0001 C CNN
+F 3 "http://www.on-shore.com/wp-content/uploads/2015/09/302-sxxx.pdf" H 5600 2800 50  0001 C CNN
+F 4 "ED10523-ND" H 5600 2800 50  0001 C CNN "Digikey"
 	1    5600 2800
 	1    0    0    -1
@@
 F 0 "J?" H 5680 3992 50  0000 L CNN
 F 1 "Conn_01x02" H 5680 3901 50  0000 L CNN
-F 2 "" H 5600 4000 50  0001 C CNN
-F 3 "~" H 5600 4000 50  0001 C CNN
+F 2 "TerminalBlock:TerminalBlock_bornier-2_P5.08mm" H 5600 4000 50  0001 C CNN
+F 3 "http://www.on-shore.com/wp-content/uploads/2015/09/ed120ds.pdf" H 5600 4000 50  0001 C CNN
+F 4 "ED1609-ND" H 5600 4000 50  0001 C CNN "Digikey"
 	1    5600 4000
 	1    0    0    -1

Commit message: Set component references
Parts:
- gave numbers to parts that had none: 2
Changed lines of the file:
@@
 GNDPWR
 $Comp
-L Connector_Generic:Conn_02x08_Odd_Even J?
+L Connector_Generic:Conn_02x08_Odd_Even J501
 U 1 1 5A7A474C
 P 5600 2800
-F 0 "J?" H 5650 3317 50  0000 C CNN
+F 0 "J501" H 5650 3317 50  0000 C CNN
 F 1 "Conn_02x08_Odd_Even" H 5650 3226 50  0000 C CNN
 F 2 "Connector_PinHeader_1.27mm:PinHeader_2x08_P1.27mm_Vertical" H 5600 2800 50  0001 C CNN
@@
 	6400 3200 5900 3200
 $Comp
-L Connector_Generic:Conn_01x02 J?
+L Connector_Generic:Conn_01x02 J502
 U 1 1 5A7F6FB6
 P 5600 4000
-F 0 "J?" H 5680 3992 50  0000 L CNN
+F 0 "J502" H 5680 3992 50  0000 L CNN
 F 1 "Conn_01x02" H 5680 3901 50  0000 L CNN
 F 2 "TerminalBlock:TerminalBlock_bornier-2_P5.08mm" H 5600 4000 50  0001 C CNN

Commit message: Spark output connector
Parts:
- added JJ503, JJ504: Conn_01x02, TerminalBlock:TerminalBlock_bornier-2_P5.08mm, symbol Connector_Generic:Conn_01x02
Connections:
- net labels added: Spark_Output
- wire segments 25 -> 29
Changed lines of the file:
@@
 Wire Wire Line
 	5400 4100 5100 4100
+$Comp
+L Connector_Generic:Conn_01x02 JJ503
+U 1 1 5A805502
+P 5600 4700
+F 0 "JJ503" H 5680 4692 50  0000 L CNN
+F 1 "Conn_01x02" H 5680 4601 50  0000 L CNN
+F 2 "TerminalBlock:TerminalBlock_bornier-2_P5.08mm" H 5600 4700 50  0001 C CNN
+F 3 "http://www.on-shore.com/wp-content/uploads/2015/09/ed120ds.pdf" H 5600 4700 50  0001 C CNN
+F 4 "ED1609-ND" H 5600 4700 50  0001 C CNN "Digikey"
+	1    5600 4700
+	1    0    0    -1
+$EndComp
+$Comp
+L Connector_Generic:Conn_01x02 JJ504
+U 1 1 5A805C17
+P 5600 5050
+F 0 "JJ504" H 5680 5042 50  0000 L CNN
+F 1 "Conn_01x02" H 5680 4951 50  0000 L CNN
+F 2 "TerminalBlock:TerminalBlock_bornier-2_P5.08mm" H 5600 5050 50  0001 C CNN
+F 3 "http://www.on-shore.com/wp-content/uploads/2015/09/ed120ds.pdf" H 5600 5050 50  0001 C CNN
+F 4 "ED1609-ND" H 5600 5050 50  0001 C CNN "Digikey"
+	1    5600 5050
+	1    0    0    -1
+$EndComp
+Text HLabel 5100 5150 0    50   Input ~ 0
+GNDPWR
+Wire Wire Line
+	5400 5150 5100 5150
+Text HLabel 5100 5050 0    50   Input ~ 0
+GNDPWR
+Wire Wire Line
+	5400 5050 5100 5050
+Text HLabel 5100 4700 0    50   Input ~ 0
+Spark_Output
+Wire Wire Line
+	5100 4700 5400 4700
+Text HLabel 5100 4800 0    50   Input ~ 0
+Spark_Output
+Wire Wire Line
+	5100 4800 5400 4800
 $EndSCHEMATC

Commit message: Plated mounting holes
Parts:
- added MK501, MK502, MK503, MK504, MK505, MK506, MK507, MK508, MK509, MK510, MK511, MK512: Mounting_Hole_PAD, MountingHole:MountingHole_5mm_Pad, symbol Mechanical:Mounting_Hole_PAD
Connections:
- wire segments 29 -> 53

Commit message: Component placement
Parts:
- J501: footprint Connector_PinHeader_1.27mm:PinHeader_2x08_P1.27mm_Vertical -> Connector_PinHeader_2.54mm:PinHeader_2x08_P2.54mm_Vertical
Changed lines of the file:
@@
 F 0 "J501" H 5650 2967 50  0000 C CNN
 F 1 "Conn_02x08_Odd_Even" H 5650 2876 50  0000 C CNN
-F 2 "Connector_PinHeader_1.27mm:PinHeader_2x08_P1.27mm_Vertical" H 5600 2450 50  0001 C CNN
+F 2 "Connector_PinHeader_2.54mm:PinHeader_2x08_P2.54mm_Vertical" H 5600 2450 50  0001 C CNN
 F 3 "http://www.on-shore.com/wp-content/uploads/2015/09/302-sxxx.pdf" H 5600 2450 50  0001 C CNN
 F 4 "ED10523-ND" H 5600 2450 50  0001 C CNN "Digikey"

Commit message: Component placement
Connections:
- wire segments 53 -> 57
Changed lines of the file:
@@
 GNDPWR
 Wire Wire Line
-	5400 4800 5100 4800
-Text HLabel 5100 4700 0    50   Input ~ 0
-GNDPWR
-Wire Wire Line
-	5400 4700 5100 4700
-Text HLabel 5100 4350 0    50   Input ~ 0
-Spark_Output
-Wire Wire Line
-	5100 4350 5400 4350
-Text HLabel 5100 4450 0    50   Input ~ 0
-Spark_Output
-Wire Wire Line
-	5100 4450 5400 4450
+	5400 4800 5300 4800
 $Comp
 L Mechanical:Mounting_Hole_PAD MK501
@@
 Wire Wire Line
 	1850 7200 2200 7200
+Text HLabel 5100 4350 0    50   Input ~ 0
+Spark_Output
+Wire Wire Line
+	5100 4350 5300 4350
+Wire Wire Line
+	5400 4450 5300 4450
+Wire Wire Line
+	5300 4450 5300 4350
+Connection ~ 5300 4350
+Wire Wire Line
+	5300 4350 5400 4350
+Wire Wire Line
+	5400 4700 5300 4700
+Wire Wire Line
+	5300 4700 5300 4800
+Connection ~ 5300 4800
+Wire Wire Line
+	5300 4800 5100 4800
 $EndSCHEMATC
