File: hardware/edm_power_board/cad/edm_power_board/edm_connectors.sch (KiCad schematic (older format))
At the start: 16 parts, among them J501 Conn_02x08_Odd_Even, J502 Conn_01x02

Commit message: Component placement
Changed lines of the file:
@@
 	1    0    0    -1
 $EndComp
+Text HLabel 6400 2550 2    50   Input ~ 0
+Output_250V_Enable
+Text HLabel 6400 2650 2    50   Input ~ 0
+Output_20V_Enable
+Text HLabel 6400 2750 2    50   Input ~ 0
+Short_Circuit
+Text HLabel 6400 2850 2    50   Input ~ 0
+Breakdown
 Text HLabel 6400 2150 2    50   Input ~ 0
-Output_250V_Enable
+Spark_Voltage_0
 Text HLabel 6400 2250 2    50   Input ~ 0
-Output_20V_Enable
+Spark_Voltage_1
 Text HLabel 6400 2350 2    50   Input ~ 0
-Short_Circuit
+Spark_Voltage_2
 Text HLabel 6400 2450 2    50   Input ~ 0
-Breakdown
-Text HLabel 6400 2550 2    50   Input ~ 0
-Spark_Voltage_0
-Text HLabel 6400 2650 2    50   Input ~ 0
-Spark_Voltage_1
-Text HLabel 6400 2750 2    50   Input ~ 0
-Spark_Voltage_2
-Text HLabel 6400 2850 2    50   Input ~ 0
 Spark_Voltage_Status
 Text HLabel 5100 2150 0    50   Input ~ 0
@@
 	5100 2150 5400 2150
 Wire Wire Line
+	5900 2550 6400 2550
+Wire Wire Line
+	6400 2650 5900 2650
+Wire Wire Line
+	5900 2750 6400 2750
+Wire Wire Line
+	6400 2850 5900 2850
+Wire Wire Line
 	5900 2150 6400 2150
 Wire Wire Line
@@
 Wire Wire Line
 	6400 2450 5900 2450
-Wire Wire Line
-	5900 2550 6400 2550
-Wire Wire Line
-	6400 2650 5900 2650
-Wire Wire Line
-	5900 2750 6400 2750
-Wire Wire Line
-	6400 2850 5900 2850
 $Comp
 L Connector_Generic:Conn_01x02 J502

Commit message: Routing
Changed lines of the file:
@@
 Comment4 ""
 $EndDescr
+Text HLabel 5100 3750 0    50   Input ~ 0
++24V
 Text HLabel 5100 3650 0    50   Input ~ 0
-+24V
-Text HLabel 5100 3750 0    50   Input ~ 0
 GNDPWR
 $Comp
@@
 $EndComp
 Wire Wire Line
-	5100 3650 5400 3650
+	5100 3750 5400 3750
 Wire Wire Line
-	5400 3750 5100 3750
+	5400 3650 5100 3650
 $Comp
 L Connector_Generic:Conn_01x02 JJ503
