File: hardware/edm_power_board/cad/edm_power_board/edm_current_source.sch (KiCad schematic (older format))
At the start: 36 parts, among them U301 LM25085MM

Commit message: Spark voltage source
Parts:
- gave numbers to parts that had none: 35

Commit message: Assign part numbers
Parts:
- C209: footprint (none) -> Capacitor_SMD:C_0805_2012Metric; Digikey (none) -> 445-1418-1-ND
Changed lines of the file:
@@
 F 0 "C209" H 6965 3546 50  0000 L CNN
 F 1 "100n" H 6965 3455 50  0000 L CNN
-F 2 "" H 6888 3350 50  0001 C CNN
+F 2 "Capacitor_SMD:C_0805_2012Metric" H 6888 3350 50  0001 C CNN
 F 3 "~" H 6850 3500 50  0001 C CNN
+F 4 "445-1418-1-ND" H 6850 3500 50  0001 C CNN "Digikey"
 	1    6850 3500
 	1    0    0    -1

Commit message: Set part numbers
Parts:
- removed C204: 220p, symbol Device:C
- removed R213, R214, R219: 1k, symbol Device:R
- removed U201: LMV321, symbol Amplifier_Operational:LMV321
- added C205: 220p, Resistor_SMD:R_0805_2012Metric, symbol Device:C
- added R202, R203: 27k, Resistor_SMD:R_0805_2012Metric, symbol Device:R
- added R217, R220, R221: 1k, Resistor_SMD:R_0805_2012Metric, symbol Device:R
- added RV201: 50k, Potentiometer_SMD:Potentiometer_Bourns_3314G_Horizontal, symbol Device:POT
- added U201: LM358, Package_SO:SOIC-8_3.9x4.9mm_P1.27mm, symbol Amplifier_Operational:LM358
- C201: footprint (none) -> Resistor_SMD:R_0805_2012Metric; Digikey (none) -> 311-1115-1-ND
- C202: value 1u -> 100n; footprint (none) -> Capacitor_SMD:C_0805_2012Metric; Digikey (none) -> 445-1418-1-ND
- C203: footprint (none) -> Capacitor_SMD:CP_Elec_5x5.3; Digikey (none) -> PCE4240CT-ND
- C204: renamed from C205; value 1u -> 100n; footprint (none) -> Capacitor_SMD:C_0805_2012Metric; Digikey (none) -> 1276-6813-1-ND
- C206: footprint (none) -> Capacitor_SMD:C_0805_2012Metric; Digikey (none) -> 490-1664-1-ND
- C207: footprint (none) -> Capacitor_SMD:C_0805_2012Metric; Digikey (none) -> 1276-1074-1-ND
- C208: footprint (none) -> Capacitor_SMD:C_0805_2012Metric; Digikey (none) -> 399-1147-1-ND
- C210: footprint (none) -> Capacitor_SMD:C_0805_2012Metric; Digikey (none) -> 311-1131-1-ND
- C211: footprint (none) -> Capacitor_SMD:CP_Elec_6.3x5.3; Digikey (none) -> PCE4209CT-ND
- D201: value TL431DBZ -> TL431AIDBZR; Digikey (none) -> 296-17329-1-ND
- D202: Digikey (none) -> 1655-1739-1-ND
- L201: footprint (none) -> Inductor_SMD:L_Wuerth_HCI-2212; Digikey (none) -> 732-4233-1-ND
- Q201: Digikey (none) -> SUD19P06-60-GE3CT-ND
- R201: value 18k -> 27k; footprint (none) -> Resistor_SMD:R_0805_2012Metric; Digikey (none) -> 311-27.0KCRCT-ND
- R204: renamed from R202; value 18k -> 4k7; footprint (none) -> Resistor_SMD:R_0805_2012Metric; Digikey (none) -> 311-4.70KCRCT-ND
- R205: renamed from R203; value 245k -> 243k; footprint (none) -> Resistor_SMD:R_0805_2012Metric; Digikey (none) -> YAG1838CT-ND
- R206: renamed from R204; footprint (none) -> Resistor_SMD:R_0805_2012Metric; Digikey (none) -> 311-10.0CRCT-ND
- R207: renamed from R205; value 25k -> 27k; footprint (none) -> Resistor_SMD:R_0805_2012Metric; Digikey (none) -> 311-27.0KCRCT-ND
- R208: renamed from R206; value 5k -> 4k7; footprint (none) -> Resistor_SMD:R_0805_2012Metric; Digikey (none) -> 311-4.70KCRCT-ND
- R209: renamed from R207; footprint (none) -> Resistor_SMD:R_0805_2012Metric; Digikey (none) -> 311-100CRCT-ND
- R210: renamed from R208; value 6k4 -> 6k34; footprint (none) -> Resistor_SMD:R_0805_2012Metric; Digikey (none) -> 311-6.34KCRCT-ND
- R211: renamed from R209; footprint (none) -> Resistor_SMD:R_2512_6332Metric; Digikey (none) -> CRA2512-FZ-R010ELFCT-ND
- R212: renamed from R210; footprint (none) -> Resistor_SMD:R_0805_2012Metric; Digikey (none) -> 311-47.0KCRCT-ND
- R213: renamed from R211; footprint (none) -> Resistor_SMD:R_0805_2012Metric; Digikey (none) -> 311-15.0KCRCT-ND
- R214: renamed from R212; footprint (none) -> Resistor_SMD:R_0805_2012Metric; Digikey (none) -> 311-1.00KCRCT-ND
- R215, R216, R218: footprint (none) -> Resistor_SMD:R_0805_2012Metric; Digikey (none) -> 311-1.00KCRCT-ND
- R219: renamed from R217; footprint (none) -> Resistor_SMD:R_Stackpole_CSSH2728_4-100m; Digikey (none) -> CSSH2728FT20L0CT-ND
- U202: renamed from U301; Digikey (none) -> LM25085MM/NOPBCT-ND
Connections:
- wire segments 131 -> 142

Commit message: PCB Outline
Parts:
- U202: footprint Package_SSOP:MSOP-8_3x3mm_P0.65mm -> Package_SO:MSOP-8_3x3mm_P0.65mm
Changed lines of the file:
@@
 F 0 "U202" H 4550 2867 50  0000 C CNN
 F 1 "LM25085MM" H 4550 2776 50  0000 C CNN
-F 2 "Package_SSOP:MSOP-8_3x3mm_P0.65mm" H 4600 1850 50  0001 L CIN
+F 2 "Package_SO:MSOP-8_3x3mm_P0.65mm" H 4600 1850 50  0001 L CIN
 F 3 "http://www.ti.com/lit/ds/symlink/lm25085.pdf" H 4550 2300 50  0001 C CNN
 F 4 "LM25085MM/NOPBCT-ND" H 4550 2300 50  0001 C CNN "Digikey"

Commit message: Plated mounting holes
Connections:
- net labels added: CS_1, CS_1+, CS_1-, CS_2, CS_2+, CS_2-, CS_3, CS_4, CS_ADJ, CS_FB, CS_ISEN, CS_NC1, CS_NC2, CS_OUT, CS_PGATE, CS_QD, CS_QD1, CS_QS, CS_RT, CS_VCC
Changed lines of the file:
@@
 L Device:R R212
 U 1 1 5A720D60
-P 6750 2950
-F 0 "R212" H 6820 2996 50  0000 L CNN
-F 1 "47k" H 6820 2905 50  0000 L CNN
-F 2 "Resistor_SMD:R_0805_2012Metric" V 6680 2950 50  0001 C CNN
-F 3 "~" H 6750 2950 50  0001 C CNN
-F 4 "311-47.0KCRCT-ND" H 6750 2950 50  0001 C CNN "Digikey"
-	1    6750 2950
+P 6700 2950
+F 0 "R212" H 6770 2996 50  0000 L CNN
+F 1 "47k" H 6770 2905 50  0000 L CNN
+F 2 "Resistor_SMD:R_0805_2012Metric" V 6630 2950 50  0001 C CNN
+F 3 "~" H 6700 2950 50  0001 C CNN
+F 4 "311-47.0KCRCT-ND" H 6700 2950 50  0001 C CNN "Digikey"
+	1    6700 2950
 	0    1    1    0
 $EndComp
@@
 L Device:C C210
 U 1 1 5A720E17
-P 7250 2950
-F 0 "C210" H 7365 2996 50  0000 L CNN
-F 1 "3n3" H 7365 2905 50  0000 L CNN
-F 2 "Capacitor_SMD:C_0805_2012Metric" H 7288 2800 50  0001 C CNN
-F 3 "~" H 7250 2950 50  0001 C CNN
-F 4 "311-1131-1-ND" H 7250 2950 50  0001 C CNN "Digikey"
-	1    7250 2950
+P 7300 2950
+F 0 "C210" H 7415 2996 50  0000 L CNN
+F 1 "3n3" H 7415 2905 50  0000 L CNN
+F 2 "Capacitor_SMD:C_0805_2012Metric" H 7338 2800 50  0001 C CNN
+F 3 "~" H 7300 2950 50  0001 C CNN
+F 4 "311-1131-1-ND" H 7300 2950 50  0001 C CNN "Digikey"
+	1    7300 2950
 	0    1    1    0
 $EndComp
@@
 L Device:C C209
 U 1 1 5A720E81
-P 7000 3350
-F 0 "C209" H 7115 3396 50  0000 L CNN
-F 1 "100n" H 7115 3305 50  0000 L CNN
-F 2 "Capacitor_SMD:C_0805_2012Metric" H 7038 3200 50  0001 C CNN
-F 3 "~" H 7000 3350 50  0001 C CNN
-F 4 "445-1418-1-ND" H 7000 3350 50  0001 C CNN "Digikey"
-	1    7000 3350
+P 7000 3400
+F 0 "C209" H 7115 3446 50  0000 L CNN
+F 1 "100n" H 7115 3355 50  0000 L CNN
+F 2 "Capacitor_SMD:C_0805_2012Metric" H 7038 3250 50  0001 C CNN
+F 3 "~" H 7000 3400 50  0001 C CNN
+F 4 "445-1418-1-ND" H 7000 3400 50  0001 C CNN "Digikey"
+	1    7000 3400
 	1    0    0    -1
 $EndComp
@@
 Connection ~ 6250 2750
 Wire Wire Line
-	6600 2950 6500 2950
+	6550 2950 6500 2950
 Wire Wire Line
 	6500 2950 6500 2750
@@
 	7150 2750 7500 2750
 Wire Wire Line
-	7400 2950 7500 2950
+	7450 2950 7500 2950
 Wire Wire Line
 	7500 2950 7500 2750
 Connection ~ 7500 2750
 Wire Wire Line
-	6900 2950 7000 2950
-Wire Wire Line
-	7000 3200 7000 2950
+	6850 2950 7000 2950
+Wire Wire Line
+	7000 3250 7000 2950
 Connection ~ 7000 2950
 Wire Wire Line
-	7000 2950 7100 2950
+	7000 2950 7150 2950
 Wire Wire Line
 	4950 2600 5400 2600
@@
 	5400 2600 5400 3600
 Wire Wire Line
-	7000 3600 7000 3500
+	7000 3600 7000 3550
 $Comp
 L Device:R R213
@@
 Wire Wire Line
 	8300 2850 8300 2750
-$Comp
-L power:GND #PWR0213
-U 1 1 5A72F141
-P 8300 3250
-F 0 "#PWR0213" H 8300 3000 50  0001 C CNN
-F 1 "GND" H 8305 3077 50  0000 C CNN
-F 2 "" H 8300 3250 50  0001 C CNN
-F 3 "" H 8300 3250 50  0001 C CNN
-	1    8300 3250
-	1    0    0    -1
-$EndComp
 Wire Wire Line
 	8300 3250 8300 3150
@@
 $EndComp
 Wire Wire Line
-	9500 4500 8650 4500
+	9500 4500 8350 4500
 Wire Wire Line
 	5900 4500 5900 5950
 Wire Wire Line
-	8900 4100 8650 4100
+	8900 4100 8350 4100
 Wire Wire Line
 	5700 4100 5700 5750
@@
 L Device:R R204
 U 1 1 5A7B5B19
-P 3250 4900
-F 0 "R204" H 3320 4946 50  0000 L CNN
-F 1 "4k7" H 3320 4855 50  0000 L CNN
-F 2 "Resistor_SMD:R_0805_2012Metric" V 3180 4900 50  0001 C CNN
-F 3 "~" H 3250 4900 50  0001 C CNN
-F 4 "311-4.70KCRCT-ND" H 3250 4900 50  0001 C CNN "Digikey"
-	1    3250 4900
-	0    1    1    0
-$EndComp
-Wire Wire Line
-	3350 5300 2950 5300
-Wire Wire Line
-	2950 5300 2950 4900
-Wire Wire Line
-	2950 4900 3100 4900
-Wire Wire Line
-	2950 4900 2750 4900
+P 3050 4900
+F 0 "R204" H 3120 4946 50  0000 L CNN
+F 1 "4k7" H 3120 4855 50  0000 L CNN
+F 2 "Resistor_SMD:R_0805_2012Metric" V 2980 4900 50  0001 C CNN
+F 3 "~" H 3050 4900 50  0001 C CNN
+F 4 "311-4.70KCRCT-ND" H 3050 4900 50  0001 C CNN "Digikey"
+	1    3050 4900
+	0    1    1    0
+$EndComp
+Wire Wire Line
+	3350 5300 2850 5300
+Wire Wire Line
+	2850 5300 2850 4900
+Wire Wire Line
+	2850 4900 2900 4900
+Wire Wire Line
+	2850 4900 2750 4900
 Wire Wire Line
 	2750 4900 2750 4200
-Connection ~ 2950 4900
+Connection ~ 2850 4900
 Wire Wire Line
 	2750 4200 3000 4200
@@
 L Device:R R207
 U 1 1 5A7F6636
-P 4700 3550
-F 0 "R207" H 4770 3596 50  0000 L CNN
-F 1 "27k" H 4770 3505 50  0000 L CNN
-F 2 "Resistor_SMD:R_0805_2012Metric" V 4630 3550 50  0001 C CNN
-F 3 "~" H 4700 3550 50  0001 C CNN
-F 4 "311-27.0KCRCT-ND" H 4700 3550 50  0001 C CNN "Digikey"
-	1    4700 3550
-	0    1    1    0
-$EndComp
-Wire Wire Line
-	4850 3550 5050 3550
+P 4650 3550
+F 0 "R207" H 4720 3596 50  0000 L CNN
+F 1 "27k" H 4720 3505 50  0000 L CNN
+F 2 "Resistor_SMD:R_0805_2012Metric" V 4580 3550 50  0001 C CNN
+F 3 "~" H 4650 3550 50  0001 C CNN
+F 4 "311-27.0KCRCT-ND" H 4650 3550 50  0001 C CNN "Digikey"
+	1    4650 3550
+	0    1    1    0
+$EndComp
+Wire Wire Line
+	4800 3550 5050 3550
 $Comp
 L Device:R R208
@@
 	5050 3550 5050 4000
 Wire Wire Line
-	4550 3550 4250 3550
+	4500 3550 4250 3550
 Wire Wire Line
 	4250 3550 4250 3700
@@
 $EndComp
 Wire Wire Line
-	3600 4900 3400 4900
+	3600 4900 3200 4900
 Wire Wire Line
 	3600 4100 3750 4100
@@
 L Device:R R215
 U 1 1 5A93681D
-P 8500 4100
-F 0 "R215" H 8570 4146 50  0000 L CNN
-F 1 "1k" H 8570 4055 50  0000 L CNN
-F 2 "Resistor_SMD:R_0805_2012Metric" V 8430 4100 50  0001 C CNN
-F 3 "~" H 8500 4100 50  0001 C CNN
-F 4 "311-1.00KCRCT-ND" H 8500 4100 50  0001 C CNN "Digikey"
-	1    8500 4100
+P 8200 4100
+F 0 "R215" H 8270 4146 50  0000 L CNN
+F 1 "1k" H 8270 4055 50  0000 L CNN
+F 2 "Resistor_SMD:R_0805_2012Metric" V 8130 4100 50  0001 C CNN
+F 3 "~" H 8200 4100 50  0001 C CNN
+F 4 "311-1.00KCRCT-ND" H 8200 4100 50  0001 C CNN "Digikey"
+	1    8200 4100
 	0    1    1    0
 $EndComp
@@
 L Device:R R216
 U 1 1 5A9368E8
-P 8500 4500
-F 0 "R216" H 8570 4546 50  0000 L CNN
-F 1 "1k" H 8570 4455 50  0000 L CNN
-F 2 "Resistor_SMD:R_0805_2012Metric" V 8430 4500 50  0001 C CNN
-F 3 "~" H 8500 4500 50  0001 C CNN
-F 4 "311-1.00KCRCT-ND" H 8500 4500 50  0001 C CNN "Digikey"
-	1    8500 4500
+P 8200 4500
+F 0 "R216" H 8270 4546 50  0000 L CNN
+F 1 "1k" H 8270 4455 50  0000 L CNN
+F 2 "Resistor_SMD:R_0805_2012Metric" V 8130 4500 50  0001 C CNN
+F 3 "~" H 8200 4500 50  0001 C CNN
+F 4 "311-1.00KCRCT-ND" H 8200 4500 50  0001 C CNN "Digikey"
+	1    8200 4500
 	0    1    1    0
 $EndComp
@@
 Connection ~ 5900 1500
 Wire Wire Line
-	5700 4100 8350 4100
-Wire Wire Line
-	5900 4500 8350 4500
+	5700 4100 8050 4100
+Wire Wire Line
+	5900 4500 8050 4500
 $Comp
 L Device:C C205
@@
 	0    1    1    0
 $EndComp
+Text Label 5100 2600 0    50   ~ 0
+CS_FB
+Text Label 5100 2400 0    50   ~ 0
+CS_ISEN
+Text Label 5100 2300 0    50   ~ 0
+CS_PGATE
+Text Label 5100 2200 0    50   ~ 0
+CS_ADJ
+Text Label 5950 2050 0    50   ~ 0
+CS_QS
+Text Label 6550 2750 0    50   ~ 0
+CS_QD
+Text Label 3900 2500 0    50   ~ 0
+CS_RT
+Text Label 3600 4100 0    50   ~ 0
+CS_1
+Text Label 4300 4100 0    50   ~ 0
+CS_2
+Text Label 4300 3550 0    50   ~ 0
+CS_3
+Text Label 4800 3550 0    50   ~ 0
+CS_4
+Text Label 6900 2950 0    50   ~ 0
+CS_QD1
+Text Label 7850 2750 0    50   ~ 0
+CS_OUT
+Text Label 8450 4100 0    50   ~ 0
+CS_1-
+Text Label 8450 4500 0    50   ~ 0
+CS_1+
+Text Label 7700 4100 0    50   ~ 0
+CS_2-
+Text Label 7700 4500 0    50   ~ 0
+CS_2+
+Text Label 3250 4900 0    50   ~ 0
+CS_FB
+Text Label 2050 6750 0    50   ~ 0
+CS_NC1
+Text Label 2400 7300 0    50   ~ 0
+CS_NC2
+Text Label 4950 2000 0    50   ~ 0
+CS_VCC
+$Comp
+L power:GNDPWR #PWR01
+U 1 1 5A876159
+P 8300 3250
+F 0 "#PWR01" H 8300 3050 50  0001 C CNN
+F 1 "GNDPWR" H 8300 3100 50  0000 C CNN
+F 2 "" H 8300 3200 50  0001 C CNN
+F 3 "" H 8300 3200 50  0001 C CNN
+	1    8300 3250
+	1    0    0    -1
+$EndComp
 $EndSCHEMATC

Commit message: Component placement
Connections:
- net labels added: CS_5
- net labels removed: GND
Changed lines of the file:
@@
 Wire Wire Line
 	2550 4000 3000 4000
-$Comp
-L power:GND #PWR0208
-U 1 1 5A794402
-P 3200 4500
-F 0 "#PWR0208" H 3200 4250 50  0001 C CNN
-F 1 "GND" H 3205 4327 50  0000 C CNN
-F 2 "" H 3200 4500 50  0001 C CNN
-F 3 "" H 3200 4500 50  0001 C CNN
-	1    3200 4500
-	1    0    0    -1
-$EndComp
 Wire Wire Line
 	3200 4400 3200 4500
@@
 F 3 "http://www.ti.com/lit/ds/symlink/lm2904-n.pdf" H 2750 6850 50  0001 C CNN
 	1    2750 6850
-	1    0    0    -1
-$EndComp
-$Comp
-L power:GND #PWR0203
-U 1 1 5A8203CF
-P 2000 7200
-F 0 "#PWR0203" H 2000 6950 50  0001 C CNN
-F 1 "GND" H 2005 7027 50  0000 C CNN
-F 2 "" H 2000 7200 50  0001 C CNN
-F 3 "" H 2000 7200 50  0001 C CNN
-	1    2000 7200
 	1    0    0    -1
 $EndComp
@@
 Text Label 7700 4500 0    50   ~ 0
 CS_2+
-Text Label 3250 4900 0    50   ~ 0
-CS_FB
+Text Label 3300 4900 0    50   ~ 0
+CS_5
 Text Label 2050 6750 0    50   ~ 0
 CS_NC1
@@
 	1    0    0    -1
 $EndComp
+$Comp
+L power:GNDPWR #PWR?
+U 1 1 5A8E371E
+P 3200 4500
+F 0 "#PWR?" H 3200 4300 50  0001 C CNN
+F 1 "GNDPWR" H 3200 4350 50  0000 C CNN
+F 2 "" H 3200 4450 50  0001 C CNN
+F 3 "" H 3200 4450 50  0001 C CNN
+	1    3200 4500
+	1    0    0    -1
+$EndComp
+$Comp
+L power:GNDPWR #PWR?
+U 1 1 5A8E3779
+P 2000 7200
+F 0 "#PWR?" H 2000 7000 50  0001 C CNN
+F 1 "GNDPWR" H 2000 7050 50  0000 C CNN
+F 2 "" H 2000 7150 50  0001 C CNN
+F 3 "" H 2000 7150 50  0001 C CNN
+	1    2000 7200
+	1    0    0    -1
+$EndComp
