File: hardware/edm_power_board/cad/edm_power_board/edm_spark_output.sch (KiCad schematic (older format))
At the start: 7 parts

Commit message: Spark output
Parts:
- added C? (x2): 1u, symbol Device:C
- added C? (x7): 100n, symbol Device:C
- added D? (x2): D, symbol Device:D
- added D? (x2): D_Schottky, symbol Device:D_Schottky
- added D? (x2): D_Zener, symbol Device:D_Zener
- added R? (x18): R, symbol Device:R
- added U?: Si8642BB-B-IS, Package_SO:SOIC-16W_7.5x10.3mm_P1.27mm, symbol Isolator:Si8642BB-B-IS
- added U? (x2): LM311, symbol Comparator:LM311
- added U?: FAN7371, Package_SO:SOIC-8_3.9x4.9mm_P1.27mm, symbol Driver_FET:FAN7371
- C?: value C -> 330n
- C?: value C -> 100n
- C?: value C -> 1u
Connections:
- net labels added: +12V, Breakdown, Output_20V_Enable, Output_250V_Enable, Short_Circuit, Spark_Output
- wire segments 17 -> 182
Other:
- moved on the sheet: Q?, U?

Commit message: Assign part numbers
Parts:
- removed C? (x5): 100n, symbol Device:C
- removed D?: D, symbol Device:D
- removed D?: D_Zener, symbol Device:D_Zener
- removed D?: D_Schottky, symbol Device:D_Schottky
- removed R? (x3): R, symbol Device:R
- removed U?: LM311, symbol Comparator:LM311
- removed U?: L78L12_SO8, Package_SO:SOIC-8_3.9x4.9mm_P1.27mm, symbol Regulator_Linear:L78L12_SO8
- added C? (x7): 100n, Capacitor_SMD:C_0805_2012Metric, symbol Device:C
- added D?: VS-15EWL06FNTR-M3, Package_TO_SOT_SMD:TO-252-2, symbol Device:D_Schottky
- added D?: RS1MTR, Diode_SMD:D_SMA, symbol Device:D
- added D?: 4V7, Diode_SMD:D_SOD-123, symbol Device:D_Zener
- added R? (x2): 47R, symbol Device:R
- added R?: 93k1, symbol Device:R
- added R? (x2): 10k, symbol Device:R
- added RV?: 250k, symbol Device:POT
- added RV?: POT, symbol Device:POT
- added U?: LM311, Package_SO:SOIC-8_3.9x4.9mm_P1.27mm, symbol Comparator:LM311
- added U?: L7815, Package_TO_SOT_SMD:TO-263-2, symbol Regulator_Linear:L7815
- C? (x2): value 1u -> 470n
- C? (x2): value 100n -> 10u
- C?: footprint (none) -> Capacitor_SMD:C_0805_2012Metric; Digikey (none) -> 445-1418-1-ND
- D?: value D -> RS1MTR; footprint (none) -> Diode_SMD:D_SMA; Digikey (none) -> 1655-1501-1-ND; Vf (none) -> 1,3V @ 1A; Vr (none) -> 1000V; trr (none) -> 500ns
- D?: value D_Schottky -> VS-15EWL06FNTR-M3; footprint (none) -> Package_TO_SOT_SMD:TO-252-2; Digikey (none) -> VS-15EWL06FNTR-M3CT-ND; Io (none) -> 15A; Vf (none) -> 1.05V @ 15A; Vr (none) -> 600V
- D?: value D_Zener -> 4V7; footprint (none) -> Diode_SMD:D_SOD-123; Digikey (none) -> BZT52C4V7-13FDICT-ND; Mfg part (none) -> BZT52C4V7-13-F
- R? (x4): value R -> 5R
- R? (x2): value R -> 4k7
- R? (x2): value R -> 21k
- R? (x3): value R -> 27k
- R?: value R -> 84k5
- R? (x3): value R -> 93k1
- U?: Digikey (none) -> SI8642BB-B-IS-ND
- U?: footprint (none) -> Package_SO:SOIC-8_3.9x4.9mm_P1.27mm; Digikey (none) -> LM311MX/NOPBCT-ND
- U? (x2): Digikey (none) -> FAN7371MXDKR-ND; Mouser (none) -> 512-FAN7371MX
Connections:
- net labels added: +15V
- net labels removed: +12V
- wire segments 182 -> 198
Other:
- note added: "2.5V"
- note added: "3.8V"
- note added: "30V"
- note added: "5V"

Commit message: Set component references
Parts:
- C607, C614: renamed from C?; footprint (none) -> Capacitor_SMD:C_0805_2012Metric; Digikey (none) -> 1276-1074-1-ND
- Q601: renamed from Q?; Digikey (none) -> IPD50R3K0CEAUMA1CT-ND
- Q602: renamed from Q?; Digikey (none) -> IPD50R380CEAUMA1CT-ND; Farnell (none) -> 2709943; Mouser (none) -> 726-IPD50R380CEAUMA1
- RV601: renamed from RV?; value POT -> 50k; footprint (none) -> Potentiometer_SMD:Potentiometer_Bourns_3314G_Horizontal; Digikey (none) -> 3314G-503ECT-ND
- RV602: renamed from RV?; footprint (none) -> Potentiometer_SMD:Potentiometer_Bourns_3314G_Horizontal; Digikey (none) -> 3314G-254ECT-ND
- gave numbers to parts that had none: 44

Commit message: Set part numbers
Parts:
- C601: footprint (none) -> Capacitor_SMD:C_0805_2012Metric; Digikey (none) -> 1276-6813-1-ND
- C604: footprint (none) -> Capacitor_SMD:C_0805_2012Metric; Digikey (none) -> 1276-1066-1-ND
- C606, C609: footprint (none) -> Capacitor_SMD:CP_Elec_6.3x5.3; Digikey (none) -> PCE4209CT-ND
- R601, R604, R605, R609: value 5R -> 4R99; footprint (none) -> Resistor_SMD:R_0805_2012Metric; Digikey (none) -> 311-4.99CRCT-ND
- R602, R607: footprint (none) -> Resistor_SMD:R_0805_2012Metric; Digikey (none) -> 311-47.0CRCT-ND
- R603, R608: footprint (none) -> Resistor_SMD:R_0805_2012Metric; Digikey (none) -> 311-4.70KCRCT-ND
- R606, R615: footprint (none) -> Resistor_SMD:R_0805_2012Metric; Digikey (none) -> 311-21.0KCRCT-ND
- R610, R616, R617: footprint (none) -> Resistor_SMD:R_0805_2012Metric; Digikey (none) -> 311-27.0KCRCT-ND
- R611: footprint (none) -> Resistor_SMD:R_0805_2012Metric; Digikey (none) -> 311-84.5KCRCT-ND
- R612, R618: footprint (none) -> Resistor_SMD:R_0805_2012Metric; Digikey (none) -> YAG1763CT-ND
- R613, R614, R619, R620: footprint (none) -> Resistor_SMD:R_0805_2012Metric; Digikey (none) -> 311-93.1KCRCT-ND

Commit message: Add input capacitors to spark
Parts:
- C604: Digikey 1276-1066-1-ND -> 587-2910-1-ND
Changed lines of the file:
@@
 F 2 "Capacitor_SMD:C_0805_2012Metric" H 3688 6800 50  0001 C CNN
 F 3 "~" H 3650 6950 50  0001 C CNN
-F 4 "1276-1066-1-ND" H 3650 6950 50  0001 C CNN "Digikey"
+F 4 "587-2910-1-ND" H 3650 6950 50  0001 C CNN "Digikey"
 	1    3650 6950
 	1    0    0    -1

Commit message: Component placement
Connections:
- net labels added: +20V_Out, +250V_Out, HV_ENA, HV_ENB, HV_VB, HV_VS, LV_ENA, LV_ENB, LV_VB, LV_VS
Changed lines of the file:
@@
 	-1   0    0    1
 $EndComp
+Text Label 5000 1650 0    50   ~ 0
++250V_Out
+Text Label 7300 1650 0    50   ~ 0
++20V_Out
+Text Label 6200 2850 0    50   ~ 0
+LV_ENA
+Text Label 7000 2350 1    50   ~ 0
+LV_ENB
+Text Label 4700 2350 1    50   ~ 0
+HV_ENB
+Text Label 3900 2850 0    50   ~ 0
+HV_ENA
+Text Label 3900 2650 0    50   ~ 0
+HV_VB
+Text Label 3900 3050 0    50   ~ 0
+HV_VS
+Text Label 6200 3050 0    50   ~ 0
+LV_VS
+Text Label 6200 2650 0    50   ~ 0
+LV_VB
+Text Label 9100 1650 0    50   ~ 0
+Spark_Output
 $EndSCHEMATC

Commit message: Component placement
Parts:
- added D607: RS1MTR, Diode_SMD:D_SMA, symbol Device:D
- added R621, R622: 21k, Resistor_SMD:R_0805_2012Metric, symbol Device:R
Connections:
- wire segments 198 -> 205
Other:
- note added: "4V"
- note removed: "5V"
Changed lines of the file:
@@
 Wire Wire Line
 	10700 3550 8850 3550
-Wire Wire Line
-	8850 3550 8850 1650
 Connection ~ 8850 1650
 Wire Wire Line
@@
 Spark_Output
 Wire Wire Line
-	8850 1650 9900 1650
+	8850 1650 8950 1650
 Wire Wire Line
 	3900 2850 4300 2850
@@
 30V
 Text Notes 10750 3700 0    50   ~ 0
-5V
+4V
 $Comp
 L Device:C C605
@@
 Text Label 9100 1650 0    50   ~ 0
 Spark_Output
+$Comp
+L Device:D D607
+U 1 1 5A81E29E
+P 9200 2500
+F 0 "D607" V 9246 2421 50  0000 R CNN
+F 1 "RS1MTR" V 9155 2421 50  0000 R CNN
+F 2 "Diode_SMD:D_SMA" H 9200 2500 50  0001 C CNN
+F 3 "http://www.smc-diodes.com/propdf/RS1A-RS1M%20N0988%20REV.B.pdf" H 9200 2500 50  0001 C CNN
+F 4 "1655-1501-1-ND" V 9200 2500 50  0001 C CNN "Digikey"
+F 5 "500ns" V 9200 2500 50  0001 C CNN "trr"
+F 6 "1,3V @ 1A" V 9200 2500 50  0001 C CNN "Vf"
+F 7 "1000V" V 9200 2500 50  0001 C CNN "Vr"
+	1    9200 2500
+	1    0    0    -1
+$EndComp
+$Comp
+L Device:R R621
+U 1 1 5A81E7BE
+P 9600 2500
+F 0 "R621" H 9530 2454 50  0000 R CNN
+F 1 "21k" H 9530 2545 50  0000 R CNN
+F 2 "Resistor_SMD:R_0805_2012Metric" V 9530 2500 50  0001 C CNN
+F 3 "~" H 9600 2500 50  0001 C CNN
+F 4 "311-21.0KCRCT-ND" H 9600 2500 50  0001 C CNN "Digikey"
+	1    9600 2500
+	0    -1   -1   0
+$EndComp
+$Comp
+L Device:R R622
+U 1 1 5A827E7D
+P 10000 2500
+F 0 "R622" H 9930 2454 50  0000 R CNN
+F 1 "21k" H 9930 2545 50  0000 R CNN
+F 2 "Resistor_SMD:R_0805_2012Metric" V 9930 2500 50  0001 C CNN
+F 3 "~" H 10000 2500 50  0001 C CNN
+F 4 "311-21.0KCRCT-ND" H 10000 2500 50  0001 C CNN "Digikey"
+	1    10000 2500
+	0    -1   -1   0
+$EndComp
+$Comp
+L power:+5V #PWR0629
+U 1 1 5A82849A
+P 10250 2400
+F 0 "#PWR0629" H 10250 2250 50  0001 C CNN
+F 1 "+5V" H 10265 2573 50  0000 C CNN
+F 2 "" H 10250 2400 50  0001 C CNN
+F 3 "" H 10250 2400 50  0001 C CNN
+	1    10250 2400
+	1    0    0    -1
+$EndComp
+Wire Wire Line
+	10150 2500 10250 2500
+Wire Wire Line
+	10250 2500 10250 2400
+Wire Wire Line
+	9750 2500 9850 2500
+Wire Wire Line
+	9450 2500 9350 2500
+Wire Wire Line
+	8950 2500 8950 1650
+Wire Wire Line
+	8850 1650 8850 3550
+Connection ~ 8950 1650
+Wire Wire Line
+	8950 1650 9900 1650
+Wire Wire Line
+	8950 2500 9050 2500
 $EndSCHEMATC

Commit message: Component placement
Parts:
- added C615: 100n, Capacitor_SMD:C_0805_2012Metric, symbol Device:C
- added D608: 1.5SMC400CA, Diode_SMD:D_SMC, symbol Device:D_Zener
Connections:
- wire segments 205 -> 210
Other:
- moved on the sheet: U602
