File: hardware/edm_power_board/cad/edm_power_board/edm_power_board.kicad_pcb (KiCad board)
At the start: 4 copper layers, 240 x 100 mm, 153 parts, among them J501 Conn_02x08_Odd_Even, J502 Conn_01x02, Q201 SUD19P06-60, Q301 BSS214NW, Q302 BSC13DN30NSFD, Q303 BSS214NW, Q304 BSS214NW, Q601 IPD50R3K0CE, Q602 IPD50R380CE, U201 LM358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

Commit message: Component placement
Parts:
- J501: footprint Connector_PinHeader_1.27mm:PinHeader_2x08_P1.27mm_Vertical -> Connector_PinHeader_2.54mm:PinHeader_2x08_P2.54mm_Vertical
- L301: footprint Inductor_SMD:L_12x12mm_H8mm -> Inductor_SMD:L_Pulse_PA4320
- moved D602 196.8 mm to (159.4, -60.1)
- moved Q601 184.6 mm to (171.9, -60.1)
- moved R603 177.2 mm to (172.0, -50.5)
- moved U601 176.7 mm to (118.0, -19.6), turned to 180 degrees
- moved R602 175.9 mm to (172.0, -47.7), turned to 180 degrees
- moved C611 175.5 mm to (166.8, -45.1)
- moved U603 172.5 mm to (166.8, -50.5), turned to 90 degrees
- moved C607 167.6 mm to (158.6, -52.3), turned to 90 degrees
- moved R604 166.1 mm to (172.0, -53.2), turned to 180 degrees
- moved R601 162.8 mm to (158.6, -48.6), turned to 270 degrees
- moved D601 162.5 mm to (161.8, -50.5), turned to 270 degrees
- moved U602 157.7 mm to (120.9, -50.9)
- moved U605 150.0 mm to (99.9, -15.1)
- moved C610 149.5 mm to (106.6, -13.3)
- moved U606 146.4 mm to (100.0, -27.8)
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Connections:
- net Net-(C607-Pad1) renamed /Spark Output/HV_VB
- net Net-(C607-Pad2) renamed /Spark Output/HV_VS
- net Net-(C614-Pad1) renamed /Spark Output/LV_VB
- net Net-(C614-Pad2) renamed /Spark Output/LV_VS
- net Net-(D602-Pad2) renamed /Spark Output/+250V_Out
- net Net-(D605-Pad2) renamed /Spark Output/+20V_Out
- net Net-(Q601-Pad1) renamed /Spark Output/HV_ENB
- net Net-(Q602-Pad1) renamed /Spark Output/LV_ENB
- net Net-(R602-Pad2) renamed /Spark Output/HV_ENA
- net Net-(R607-Pad2) renamed /Spark Output/LV_ENA
- R203 pad 2: GND -> GNDPWR
- R204 pad 1: /Current Source/CS_FB -> /Current Source/CS_5
- RV201 pad 2: /Current Source/CS_FB -> /Current Source/CS_5
- U201 pad 4: GND -> GNDPWR

Commit message: Component placement
Parts:
- added D607: RS1MTR, Diode_SMD:D_SMA, F.Cu at (68.5, -10.8)
- added R621: 21k, Resistor_SMD:R_0805_2012Metric, F.Cu at (75.0, -10.8)
- added R622: 21k, Resistor_SMD:R_0805_2012Metric, F.Cu at (79.4, -10.8)
- moved C303 8.90 mm to (168.4, -22.7)
- moved C308 8.70 mm to (182.7, -22.7)
- moved C613 3.31 mm to (82.8, -53.8)
- moved C614 3.31 mm to (75.8, -45.5)
- moved R605 3.31 mm to (79.5, -45.5)
- moved R607 3.31 mm to (74.8, -58.9)
- moved D605 3.31 mm to (68.4, -60.3)
- moved R608 3.31 mm to (77.2, -58.9)
- moved R609 3.31 mm to (79.6, -58.9)
- moved D603 3.31 mm to (77.6, -48.7)
- moved Q602 3.31 mm to (68.3, -47.6)
- moved U604 3.31 mm to (77.5, -53.8)
- moved J501 2.49 mm to (136.3, -9.26)
- moved C603 1.52 mm to (124.6, -22.7)
- moved U601 1.52 mm to (117.4, -18.2)
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Connections:
- D602 pad 1: /Spark Output/Spark_Output -> /Connectors/Spark_Output
- D605 pad 1: /Spark Output/Spark_Output -> /Connectors/Spark_Output
- R613 pad 2: /Spark Output/Spark_Output -> /Connectors/Spark_Output
- R619 pad 2: /Spark Output/Spark_Output -> /Connectors/Spark_Output

Commit message: Component placement
Parts:
- added C615: 100n, Capacitor_SMD:C_0805_2012Metric, F.Cu at (59.0, -18.0)
- added D608: 1.5SMC400CA, Diode_SMD:D_SMC, F.Cu at (205.6, -69.0)
- moved D607 148.6 mm to (217.0, -16.0), turned to 180 degrees
- moved D605 143.8 mm to (210.1, -35.8), turned to 180 degrees
- moved R607 138.3 mm to (208.7, -24.0), turned to 180 degrees
- moved R619 136.2 mm to (210.0, -7.00), turned to 0 degrees
- moved R613 135.5 mm to (210.0, -10.0), turned to 0 degrees
- moved R621 135.2 mm to (210.0, -16.0), turned to 180 degrees
- moved R608 134.8 mm to (208.7, -29.0), turned to 180 degrees
- moved R609 133.0 mm to (208.7, -26.6), turned to 180 degrees
- moved Q602 129.6 mm to (197.4, -35.9), turned to 180 degrees
- moved U604 129.0 mm to (203.7, -26.7), turned to 90 degrees
- moved R620 126.9 mm to (205.0, -7.00), turned to 0 degrees
- moved R614 126.1 mm to (205.0, -10.0), turned to 0 degrees
- moved R622 125.8 mm to (205.0, -16.0), turned to 180 degrees
- moved C613 125.0 mm to (203.6, -21.4), turned to 0 degrees
- moved C303 124.4 mm to (44.0, -22.0)
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Connections:
- J501 pad 10: /Connectors/Spark_Voltage_0 -> /Connectors/Output_250V_Enable
- J501 pad 12: /Connectors/Spark_Voltage_1 -> /Connectors/Output_20V_Enable
- J501 pad 14: /Connectors/Spark_Voltage_2 -> /Connectors/Short_Circuit
- J501 pad 16: /Connectors/Spark_Voltage_Status -> /Connectors/Breakdown
- J501 pad 2: /Connectors/Output_250V_Enable -> /Connectors/Spark_Voltage_0
- J501 pad 4: /Connectors/Output_20V_Enable -> /Connectors/Spark_Voltage_1
- J501 pad 6: /Connectors/Short_Circuit -> /Connectors/Spark_Voltage_2
- J501 pad 8: /Connectors/Breakdown -> /Connectors/Spark_Voltage_Status
Routing:
- added copper zone on F.Cu, net /Connectors/Spark_Output
- added copper zone on F.Cu, net /Current Source/+20V
- added copper zone on F.Cu, net /Spark Output/+250V
- added copper zone on In1.Cu, net GNDPWR
Other:
- outline, holes or cut-outs redrawn

Commit message: Routing
Parts:
- moved D202 1.32 mm to (146.8, -63.0)
- moved Q201 0.76 mm to (145.0, -56.2), turned to 0 degrees
- moved R209 0.61 mm to (149.5, -50.0)
Connections:
- net Net-(C309-Pad1) renamed /Spark Voltage Source/VS_VCC
- net Net-(C310-Pad1) renamed /Spark Voltage Source/VS_FB
- net Net-(C311-Pad2) renamed /Spark Voltage Source/VS_COMP
- net Net-(C312-Pad1) renamed /Spark Voltage Source/VS_CS2
- net Net-(D302-Pad2) renamed /Spark Voltage Source/VS_QD
- net Net-(Q302-Pad1) renamed /Spark Voltage Source/VS_QS
- net Net-(Q302-Pad4) renamed /Spark Voltage Source/VS_OUT
- net Net-(R301-Pad2) renamed /Spark Voltage Source/VS_UVLO
- net Net-(R303-Pad1) renamed /Spark Voltage Source/VS_RT
- net Net-(R309-Pad2) renamed /Spark Voltage Source/VS_CS
- J502 pad 1: +24V -> GNDPWR
- J502 pad 2: GNDPWR -> +24V
Routing:
- net GNDPWR: track 0.00 -> 64.1 mm, vias 0 -> 36
- net /Current Source/CS_PGATE: track 0.00 -> 26.7 mm, vias 0 -> 2
- net /Current Source/CS_2+: track 0.00 -> 23.6 mm
- net /Current Source/CS_1: track 0.00 -> 21.6 mm
- net /Current Source/CS_OUT: track 0.00 -> 19.3 mm
- net +24V: track 0.00 -> 18.4 mm, vias 0 -> 10
- net /Current Source/CS_4: track 0.00 -> 16.4 mm, vias 0 -> 2
- net /Current Source/CS_2-: track 0.00 -> 14.4 mm
- net /Current Source/CS_QD: track 0.00 -> 13.9 mm, vias 0 -> 2
- net Net-(C306-Pad1): track 0.00 -> 9.75 mm
- net /Current Source/CS_1-: track 0.00 -> 9.08 mm
- net /Current Source/CS_1+: track 0.00 -> 8.96 mm
- net /Spark Voltage Source/VS_RT: track 0.00 -> 8.74 mm
- net /Spark Voltage Source/VS_CS: track 0.00 -> 8.46 mm
- net /Current Source/CS_NC1: track 0.00 -> 8.03 mm
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- added copper zone on F.Cu, net +24V
- added copper zone on In2.Cu, net +24V
- added copper zone on F.Cu, net /Current Source/CS_OUT
- added copper zone on F.Cu, net /Current Source/CS_QD
- added copper zone on F.Cu, net /Current Source/CS_QS
Other:
- net class Default: trace_width 0.25 -> 0.3; via_dia 0.8 -> 0.65; via_drill 0.4 -> 0.3
