File: hardware/edm_power_board/cad/edm_power_board/edm_power_board.kicad_pcb (KiCad board)
At the start: 4 copper layers, 240 x 100 mm, 158 parts, among them J501 Conn_02x08_Odd_Even, J502 Conn_01x02, Q201 SUD19P06-60, Q301 BSS214NW, Q302 BSC13DN30NSFD, Q303 BSS214NW, Q304 BSS214NW, Q601 IPD50R3K0CE, Q602 IPD50R380CE, U201 LM358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

Commit message: Routing
Parts:
- moved C313 4.78 mm to (102.0, -66.0), turned to 270 degrees
- moved C314 4.38 mm to (106.4, -66.0), turned to 270 degrees
- moved C309 0.60 mm to (99.7, -48.1)
- moved R309 0.60 mm to (103.2, -44.1)
- moved C310 0.60 mm to (103.1, -51.9)
- moved C311 0.60 mm to (99.6, -55.7)
- moved C312 0.60 mm to (99.6, -44.1)
- moved R305 0.60 mm to (99.6, -51.9)
- moved R314 0.60 mm to (103.1, -48.1)
- moved R317 0.60 mm to (103.1, -55.7)
- moved R310 0.30 mm to (94.2, -60.5)
- moved R311 0.10 mm to (94.2, -57.7)
- moved R315 0.10 mm to (102.4, -59.3)
Routing:
- net GNDPWR: track 64.1 -> 106.8 mm, vias 36 -> 63
- net /Spark Voltage Source/VS_FB: track 0.00 -> 31.9 mm
- net /Spark Output/+250V: track 0.00 -> 23.6 mm
- net /Spark Voltage Source/VS_COMP: track 0.00 -> 17.9 mm
- net /Spark Voltage Source/VS_VCC: track 0.00 -> 12.1 mm
- net /Spark Voltage Source/VS_QD: track 0.00 -> 10.8 mm
- net /Spark Voltage Source/VS_OUT: track 0.00 -> 9.17 mm
- net /Spark Voltage Source/VS_QS: track 0.00 -> 8.70 mm, vias 0 -> 2
- net /Spark Voltage Source/VS_CS2: track 0.00 -> 5.60 mm
- net Net-(R310-Pad2): track 0.00 -> 5.04 mm
- net +5V: track 0.00 -> 4.25 mm
- net Net-(Q304-Pad3): track 0.00 -> 2.83 mm
- net Net-(Q303-Pad3): track 0.00 -> 2.42 mm
- net Net-(Q301-Pad3): track 0.00 -> 1.72 mm
- net /Spark Voltage Source/VS_CS: track 8.46 -> 9.06 mm
- added copper zone on F.Cu, net /Spark Voltage Source/VS_QD
- added copper zone on F.Cu, net /Spark Voltage Source/VS_QS

Commit message: Routing
Parts:
- moved C401 1.42 mm to (107.0, -12.1)
- moved C402 1.42 mm to (95.9, -9.50)
- moved C403 1.42 mm to (95.9, -12.1)
- moved U401 1.42 mm to (101.8, -11.1)
- moved R608 0.19 mm to (208.7, -29.2)
Routing:
- net Net-(D606-Pad1): track 0.00 -> 82.9 mm
- net Net-(U601-Pad14): track 0.00 -> 70.3 mm, vias 0 -> 2
- net GNDPWR: track 106.8 -> 170.9 mm, vias 63 -> 82
- net Net-(D604-Pad1): track 0.00 -> 58.7 mm
- net +5V: track 4.25 -> 56.2 mm, vias 0 -> 2
- net Net-(U601-Pad13): track 0.00 -> 38.3 mm
- net /Spark Output/HV_ENB: track 0.00 -> 20.9 mm
- net +15V: track 0.00 -> 18.3 mm, vias 0 -> 14
- net /Spark Output/HV_VS: track 0.00 -> 16.7 mm
- net /Spark Output/LV_VS: track 0.00 -> 16.2 mm
- net /Spark Output/LV_ENB: track 0.00 -> 16.0 mm, vias 0 -> 2
- net /Spark Output/+250V_Out: track 0.00 -> 12.3 mm
- net Net-(R306-Pad2): track 0.00 -> 10.2 mm
- net /Spark Output/+20V_Out: track 0.00 -> 9.88 mm
- net Net-(D301-Pad1): track 0.00 -> 9.18 mm
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- added copper zone on In2.Cu, net +15V
- added copper zone on In2.Cu, net +5V
- added copper zone on F.Cu, net /Spark Output/+20V_Out
- added copper zone on F.Cu, net /Spark Output/+250V_Out
- added copper zone on F.Cu, net GNDPWR
Other:
- net class 2mm added: clearance 0.2, trace_width 2, via_dia 0.65, via_drill 0.3

Commit message: Routing
Routing:
- net Net-(U601-Pad14): track 70.3 -> 185.6 mm
- net Net-(U601-Pad13): track 38.3 -> 152.7 mm
- net +5V: track 56.2 -> 165.8 mm, vias 2 -> 16
- net Net-(R606-Pad1): track 0.00 -> 97.5 mm
- net Net-(R304-Pad2): track 5.42 -> 86.6 mm
- net Net-(R615-Pad1): track 0.00 -> 74.7 mm
- net Net-(Q304-Pad1): track 0.00 -> 65.1 mm
- net Net-(Q303-Pad1): track 0.00 -> 64.4 mm
- net Net-(Q301-Pad1): track 0.00 -> 63.9 mm
- net GNDPWR: track 170.9 -> 212.4 mm, vias 82 -> 108
- net /Connectors/Spark_Voltage_Status: track 0.00 -> 22.5 mm
- net /Connectors/Spark_Voltage_0: track 0.00 -> 22.3 mm
- net /Connectors/Breakdown: track 0.00 -> 22.2 mm
- net /Connectors/Output_250V_Enable: track 0.00 -> 21.2 mm
- net /Connectors/Short_Circuit: track 0.00 -> 21.0 mm
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- added copper zone on In2.Cu, net +3V3
- added copper zone on F.Cu, net /Spark Output/+24V
- added copper zone on In1.Cu, net GND
- added copper zone on In2.Cu, net GNDPWR
