File: hardware/edm_power_board/cad/edm_current_source.sch (KiCad schematic (older format))
At the start: 39 parts, among them Q201 SUD19P06-60, U201 LM358, U202 LM25085MM

Commit message: Add bleeder resistor, remove 25u capacitors
Changed lines of the file:
@@
 	3750 4100 3850 4100
 Wire Wire Line
-	3750 4600 4050 4600
+	3750 4600 4150 4600
 Wire Wire Line
-	4050 4600 4050 5300
+	4150 4600 4150 5300
 Wire Wire Line
-	4050 5300 3650 5300
+	4150 5300 3650 5300
 Connection ~ 3750 4600
 Wire Wire Line
