File: hardware/edm_power_board/cad/edm_spark_voltage_source.sch (KiCad schematic (older format))
At the start: 44 parts, among them Q301 BSS214NW, Q302 BSC13DN30NSFD, Q303 BSS214NW, Q304 BSS214NW, U301 Si8641BB-B-IS, U302 LM5022MM, U303 LM311

Commit message: Add bleeder resistor, remove 25u capacitors
Parts:
- C315, C316: value 25u -> 470n; footprint Capacitor_THT:C_Rect_L41.5mm_W20.0mm_P37.50mm_MKS4 -> Capacitor_SMD:C_1812_4532Metric; Digikey P15874-ND -> 445-13461-1-ND
- R308, R316: value 261R -> 26k1; Digikey 311-261CRCT-ND -> 311-26.1KCRCT-ND
- R313: value 523R -> 52k3; Digikey 311-523CRCT-ND -> 311-52.3KCRCT-ND
- R317: value 21k -> 2M1; Digikey 311-21.0KCRCT-ND -> 311-2.10MCRCT-ND
- R318: value 180R -> 18k; Digikey 311-180CRCT-ND -> 311-18.0KCRCT-ND
Changed lines of the file:
@@
 P 5900 3700
 F 0 "R308" H 5970 3746 50  0000 L CNN
-F 1 "261R" H 5970 3655 50  0000 L CNN
+F 1 "26k1" H 5970 3655 50  0000 L CNN
 F 2 "Resistor_SMD:R_0805_2012Metric" V 5830 3700 50  0001 C CNN
 F 3 "~" H 5900 3700 50  0001 C CNN
-F 4 "311-261CRCT-ND" H 5900 3700 50  0001 C CNN "Digikey"
+F 4 "311-26.1KCRCT-ND" H 5900 3700 50  0001 C CNN "Digikey"
 	1    5900 3700
 	1    0    0    -1
@@
 P 7700 2700
 F 0 "R317" H 7770 2746 50  0000 L CNN
-F 1 "21k" H 7770 2655 50  0000 L CNN
+F 1 "2M1" H 7770 2655 50  0000 L CNN
 F 2 "Resistor_SMD:R_0805_2012Metric" V 7630 2700 50  0001 C CNN
 F 3 "~" H 7700 2700 50  0001 C CNN
-F 4 "311-21.0KCRCT-ND" H 7700 2700 50  0001 C CNN "Digikey"
+F 4 "311-2.10MCRCT-ND" H 7700 2700 50  0001 C CNN "Digikey"
 	1    7700 2700
 	1    0    0    -1
@@
 P 6500 3700
 F 0 "R313" H 6570 3746 50  0000 L CNN
-F 1 "523R" H 6570 3655 50  0000 L CNN
+F 1 "52k3" H 6570 3655 50  0000 L CNN
 F 2 "Resistor_SMD:R_0805_2012Metric" V 6430 3700 50  0001 C CNN
 F 3 "~" H 6500 3700 50  0001 C CNN
-F 4 "311-523CRCT-ND" H 6500 3700 50  0001 C CNN "Digikey"
+F 4 "311-52.3KCRCT-ND" H 6500 3700 50  0001 C CNN "Digikey"
 	1    6500 3700
 	1    0    0    -1
@@
 P 8500 3700
 F 0 "R318" H 8570 3746 50  0000 L CNN
-F 1 "180R" H 8570 3655 50  0000 L CNN
+F 1 "18k" H 8570 3655 50  0000 L CNN
 F 2 "Resistor_SMD:R_0805_2012Metric" V 8430 3700 50  0001 C CNN
 F 3 "~" H 8500 3700 50  0001 C CNN
-F 4 "311-180CRCT-ND" H 8500 3700 50  0001 C CNN "Digikey"
+F 4 "311-18.0KCRCT-ND" H 8500 3700 50  0001 C CNN "Digikey"
 	1    8500 3700
 	1    0    0    -1
@@
 P 7500 3700
 F 0 "R316" H 7570 3746 50  0000 L CNN
-F 1 "261R" H 7570 3655 50  0000 L CNN
+F 1 "26k1" H 7570 3655 50  0000 L CNN
 F 2 "Resistor_SMD:R_0805_2012Metric" V 7430 3700 50  0001 C CNN
 F 3 "~" H 7500 3700 50  0001 C CNN
-F 4 "311-261CRCT-ND" H 7500 3700 50  0001 C CNN "Digikey"
+F 4 "311-26.1KCRCT-ND" H 7500 3700 50  0001 C CNN "Digikey"
 	1    7500 3700
 	1    0    0    -1
@@
 	8200 1800 8700 1800
 Connection ~ 8700 1800
-$Comp
-L Device:C C315
-U 1 1 5A8E5211
-P 9200 1550
-F 0 "C315" H 9315 1596 50  0000 L CNN
-F 1 "25u" H 9315 1505 50  0000 L CNN
-F 2 "Capacitor_THT:C_Rect_L41.5mm_W20.0mm_P37.50mm_MKS4" H 9238 1400 50  0001 C CNN
-F 3 "~" H 9200 1550 50  0001 C CNN
-F 4 "P15874-ND" H 9200 1550 50  0001 C CNN "Digikey"
-	1    9200 1550
-	1    0    0    -1
-$EndComp
-$Comp
-L Device:C C316
-U 1 1 5A8EE597
-P 9750 1550
-F 0 "C316" H 9865 1596 50  0000 L CNN
-F 1 "25u" H 9865 1505 50  0000 L CNN
-F 2 "Capacitor_THT:C_Rect_L41.5mm_W20.0mm_P37.50mm_MKS4" H 9788 1400 50  0001 C CNN
-F 3 "~" H 9750 1550 50  0001 C CNN
-F 4 "P15874-ND" H 9750 1550 50  0001 C CNN "Digikey"
-	1    9750 1550
-	1    0    0    -1
-$EndComp
 $Comp
 L Transistor_FET:BSS214NW Q303
@@
 Text Label 6800 1550 1    50   ~ 0
 VS_QD
+$Comp
+L Device:C C315
+U 1 1 5A84FFCC
+P 9200 1550
+F 0 "C315" H 9315 1596 50  0000 L CNN
+F 1 "470n" H 9315 1505 50  0000 L CNN
+F 2 "Capacitor_SMD:C_1812_4532Metric" H 9238 1400 50  0001 C CNN
+F 3 "~" H 9200 1550 50  0001 C CNN
+F 4 "445-13461-1-ND" H 9200 1550 50  0001 C CNN "Digikey"
+	1    9200 1550
+	1    0    0    -1
+$EndComp
+$Comp
+L Device:C C316
+U 1 1 5A85007D
+P 9750 1550
+F 0 "C316" H 9865 1596 50  0000 L CNN
+F 1 "470n" H 9865 1505 50  0000 L CNN
+F 2 "Capacitor_SMD:C_1812_4532Metric" H 9788 1400 50  0001 C CNN
+F 3 "~" H 9750 1550 50  0001 C CNN
+F 4 "445-13461-1-ND" H 9750 1550 50  0001 C CNN "Digikey"
+	1    9750 1550
+	1    0    0    -1
+$EndComp
 $EndSCHEMATC
