File: hardware/edm_power_board/cad/edm_spark_output.sch (KiCad schematic (older format))
At the start: 55 parts, among them Q601 IPD50R3K0CE, Q602 IPD50R380CE, U601 Si8642BB-B-IS, U602 L7815, U603 FAN7371, U604 FAN7371, U605 LM311, U606 LM311

Commit message: Add bleeder resistor, remove 25u capacitors
Parts:
- added R623: 21k, Resistor_SMD:R_0805_2012Metric, symbol Device:R
- R612, R618: value 10k -> 21k; Digikey YAG1763CT-ND -> 311-21.0KCRCT-ND
- R613, R614, R619, R620: value 93k1 -> 187k; Digikey 311-93.1KCRCT-ND -> 311-187KCRCT-ND
- RV601: value 50k -> 100k; Digikey 3314G-503ECT-ND -> 3314G-104ECT-ND
- RV602: value 250k -> 500k; Digikey 3314G-254ECT-ND -> 3314G-504ECT-ND
Connections:
- wire segments 210 -> 213
Changed lines of the file:
@@
 P 8200 3900
 F 0 "R613" H 8130 3854 50  0000 R CNN
-F 1 "93k1" H 8130 3945 50  0000 R CNN
+F 1 "187k" H 8130 3945 50  0000 R CNN
 F 2 "Resistor_SMD:R_0805_2012Metric" V 8130 3900 50  0001 C CNN
 F 3 "~" H 8200 3900 50  0001 C CNN
-F 4 "311-93.1KCRCT-ND" H 8200 3900 50  0001 C CNN "Digikey"
+F 4 "311-187KCRCT-ND" H 8200 3900 50  0001 C CNN "Digikey"
 	1    8200 3900
 	-1   0    0    1
@@
 P 10700 4800
 F 0 "RV602" V 10586 4800 50  0000 C CNN
-F 1 "250k" V 10495 4800 50  0000 C CNN
+F 1 "500k" V 10495 4800 50  0000 C CNN
 F 2 "Potentiometer_SMD:Potentiometer_Bourns_3314G_Horizontal" H 10700 4800 50  0001 C CNN
 F 3 "~" H 10700 4800 50  0001 C CNN
-F 4 "3314G-254ECT-ND" V 10700 4800 50  0001 C CNN "Digikey"
+F 4 "3314G-504ECT-ND" V 10700 4800 50  0001 C CNN "Digikey"
 	1    10700 4800
 	0    -1   -1   0
@@
 P 8200 4800
 F 0 "RV601" V 8086 4800 50  0000 C CNN
-F 1 "50k" V 7995 4800 50  0000 C CNN
+F 1 "100k" V 7995 4800 50  0000 C CNN
 F 2 "Potentiometer_SMD:Potentiometer_Bourns_3314G_Horizontal" H 8200 4800 50  0001 C CNN
 F 3 "~" H 8200 4800 50  0001 C CNN
-F 4 "3314G-503ECT-ND" V 8200 4800 50  0001 C CNN "Digikey"
+F 4 "3314G-104ECT-ND" V 8200 4800 50  0001 C CNN "Digikey"
 	1    8200 4800
 	0    -1   -1   0
@@
 P 8100 5250
 F 0 "R612" H 8030 5204 50  0000 R CNN
-F 1 "10k" H 8030 5295 50  0000 R CNN
+F 1 "21k" H 8030 5295 50  0000 R CNN
 F 2 "Resistor_SMD:R_0805_2012Metric" V 8030 5250 50  0001 C CNN
 F 3 "~" H 8100 5250 50  0001 C CNN
-F 4 "YAG1763CT-ND" H 8100 5250 50  0001 C CNN "Digikey"
+F 4 "311-21.0KCRCT-ND" H 8100 5250 50  0001 C CNN "Digikey"
 	1    8100 5250
 	0    -1   -1   0
@@
 P 10600 5250
 F 0 "R618" H 10530 5204 50  0000 R CNN
-F 1 "10k" H 10530 5295 50  0000 R CNN
+F 1 "21k" H 10530 5295 50  0000 R CNN
 F 2 "Resistor_SMD:R_0805_2012Metric" V 10530 5250 50  0001 C CNN
 F 3 "~" H 10600 5250 50  0001 C CNN
-F 4 "YAG1763CT-ND" H 10600 5250 50  0001 C CNN "Digikey"
+F 4 "311-21.0KCRCT-ND" H 10600 5250 50  0001 C CNN "Digikey"
 	1    10600 5250
 	0    -1   -1   0
@@
 P 8200 4300
 F 0 "R614" H 8130 4254 50  0000 R CNN
-F 1 "93k1" H 8130 4345 50  0000 R CNN
+F 1 "187k" H 8130 4345 50  0000 R CNN
 F 2 "Resistor_SMD:R_0805_2012Metric" V 8130 4300 50  0001 C CNN
 F 3 "~" H 8200 4300 50  0001 C CNN
-F 4 "311-93.1KCRCT-ND" H 8200 4300 50  0001 C CNN "Digikey"
+F 4 "311-187KCRCT-ND" H 8200 4300 50  0001 C CNN "Digikey"
 	1    8200 4300
 	-1   0    0    1
@@
 P 10700 3900
 F 0 "R619" H 10630 3854 50  0000 R CNN
-F 1 "93k1" H 10630 3945 50  0000 R CNN
+F 1 "187k" H 10630 3945 50  0000 R CNN
 F 2 "Resistor_SMD:R_0805_2012Metric" V 10630 3900 50  0001 C CNN
 F 3 "~" H 10700 3900 50  0001 C CNN
-F 4 "311-93.1KCRCT-ND" H 10700 3900 50  0001 C CNN "Digikey"
+F 4 "311-187KCRCT-ND" H 10700 3900 50  0001 C CNN "Digikey"
 	1    10700 3900
 	-1   0    0    1
@@
 P 10700 4300
 F 0 "R620" H 10630 4254 50  0000 R CNN
-F 1 "93k1" H 10630 4345 50  0000 R CNN
+F 1 "187k" H 10630 4345 50  0000 R CNN
 F 2 "Resistor_SMD:R_0805_2012Metric" V 10630 4300 50  0001 C CNN
 F 3 "~" H 10700 4300 50  0001 C CNN
-F 4 "311-93.1KCRCT-ND" H 10700 4300 50  0001 C CNN "Digikey"
+F 4 "311-187KCRCT-ND" H 10700 4300 50  0001 C CNN "Digikey"
 	1    10700 4300
 	-1   0    0    1
@@
 Connection ~ 9250 1650
 Wire Wire Line
-	9250 1650 10250 1650
+	9250 1650 10000 1650
 $Comp
 L power:GNDPWR #PWR0630
@@
 Wire Wire Line
 	5600 5500 5600 5400
+$Comp
+L Device:R R623
+U 1 1 5A860AAE
+P 10000 2050
+F 0 "R623" H 9930 2004 50  0000 R CNN
+F 1 "21k" H 9930 2095 50  0000 R CNN
+F 2 "Resistor_SMD:R_0805_2012Metric" V 9930 2050 50  0001 C CNN
+F 3 "~" H 10000 2050 50  0001 C CNN
+F 4 "311-21.0KCRCT-ND" H 10000 2050 50  0001 C CNN "Digikey"
+	1    10000 2050
+	-1   0    0    1
+$EndComp
+Wire Wire Line
+	10000 1900 10000 1650
+Connection ~ 10000 1650
+Wire Wire Line
+	10000 1650 10250 1650
+$Comp
+L power:GNDPWR #PWR0631
+U 1 1 5A895063
+P 10000 2400
+F 0 "#PWR0631" H 10000 2200 50  0001 C CNN
+F 1 "GNDPWR" H 10000 2200 50  0000 C CNN
+F 2 "" H 10000 2350 50  0001 C CNN
+F 3 "" H 10000 2350 50  0001 C CNN
+	1    10000 2400
+	1    0    0    -1
+$EndComp
+Wire Wire Line
+	10000 2400 10000 2200
 $EndSCHEMATC

Commit message: Update bleed resistor
Parts:
- added R624: 187k, Resistor_SMD:R_0805_2012Metric, symbol Device:R
- R623: value 21k -> 187k; Digikey 311-21.0KCRCT-ND -> 311-187KCRCT-ND
Connections:
- wire segments 213 -> 214
Changed lines of the file:
@@
 	6200 1650 6200 1200
 Wire Wire Line
-	6200 1200 8650 1200
-Wire Wire Line
-	8650 1200 8650 1650
-Wire Wire Line
-	8200 1650 8650 1650
-Connection ~ 8650 1650
-Wire Wire Line
-	10700 3550 8850 3550
-Connection ~ 8850 1650
+	6200 1200 8550 1200
+Wire Wire Line
+	8550 1200 8550 1650
+Wire Wire Line
+	8200 1650 8550 1650
+Connection ~ 8550 1650
+Wire Wire Line
+	10700 3550 8750 3550
+Connection ~ 8750 1650
 Wire Wire Line
 	2550 2400 2550 2200
@@
 Spark_Output
 Wire Wire Line
-	8850 1650 8950 1650
+	8750 1650 8850 1650
 Wire Wire Line
 	3900 2850 4300 2850
@@
 $EndComp
 Wire Wire Line
+	8550 1650 8650 1650
+Wire Wire Line
+	8200 3750 8200 3550
+Wire Wire Line
+	8200 3550 8650 3550
+Wire Wire Line
+	8650 3550 8650 1650
+Connection ~ 8650 1650
+Wire Wire Line
 	8650 1650 8750 1650
-Wire Wire Line
-	8200 3750 8200 3550
-Wire Wire Line
-	8200 3550 8750 3550
-Wire Wire Line
-	8750 3550 8750 1650
-Connection ~ 8750 1650
-Wire Wire Line
-	8750 1650 8850 1650
 $Comp
 L Device:D D603
@@
 L Device:D D607
 U 1 1 5A81E29E
-P 9200 3050
-F 0 "D607" V 9246 2971 50  0000 R CNN
-F 1 "RS1MTR" V 9155 2971 50  0000 R CNN
-F 2 "Diode_SMD:D_SMA" H 9200 3050 50  0001 C CNN
-F 3 "http://www.smc-diodes.com/propdf/RS1A-RS1M%20N0988%20REV.B.pdf" H 9200 3050 50  0001 C CNN
-F 4 "1655-1501-1-ND" V 9200 3050 50  0001 C CNN "Digikey"
-F 5 "500ns" V 9200 3050 50  0001 C CNN "trr"
-F 6 "1,3V @ 1A" V 9200 3050 50  0001 C CNN "Vf"
-F 7 "1000V" V 9200 3050 50  0001 C CNN "Vr"
-	1    9200 3050
+P 9400 3050
+F 0 "D607" V 9446 2971 50  0000 R CNN
+F 1 "RS1MTR" V 9355 2971 50  0000 R CNN
+F 2 "Diode_SMD:D_SMA" H 9400 3050 50  0001 C CNN
+F 3 "http://www.smc-diodes.com/propdf/RS1A-RS1M%20N0988%20REV.B.pdf" H 9400 3050 50  0001 C CNN
+F 4 "1655-1501-1-ND" V 9400 3050 50  0001 C CNN "Digikey"
+F 5 "500ns" V 9400 3050 50  0001 C CNN "trr"
+F 6 "1,3V @ 1A" V 9400 3050 50  0001 C CNN "Vf"
+F 7 "1000V" V 9400 3050 50  0001 C CNN "Vr"
+	1    9400 3050
 	1    0    0    -1
 $EndComp
@@
 L Device:R R621
 U 1 1 5A81E7BE
-P 9600 3050
-F 0 "R621" H 9530 3004 50  0000 R CNN
-F 1 "21k" H 9530 3095 50  0000 R CNN
-F 2 "Resistor_SMD:R_0805_2012Metric" V 9530 3050 50  0001 C CNN
-F 3 "~" H 9600 3050 50  0001 C CNN
-F 4 "311-21.0KCRCT-ND" H 9600 3050 50  0001 C CNN "Digikey"
-	1    9600 3050
+P 9800 3050
+F 0 "R621" H 9730 3004 50  0000 R CNN
+F 1 "21k" H 9730 3095 50  0000 R CNN
+F 2 "Resistor_SMD:R_0805_2012Metric" V 9730 3050 50  0001 C CNN
+F 3 "~" H 9800 3050 50  0001 C CNN
+F 4 "311-21.0KCRCT-ND" H 9800 3050 50  0001 C CNN "Digikey"
+	1    9800 3050
 	0    -1   -1   0
 $EndComp
@@
 L Device:R R622
 U 1 1 5A827E7D
-P 10000 3050
-F 0 "R622" H 9930 3004 50  0000 R CNN
-F 1 "21k" H 9930 3095 50  0000 R CNN
-F 2 "Resistor_SMD:R_0805_2012Metric" V 9930 3050 50  0001 C CNN
-F 3 "~" H 10000 3050 50  0001 C CNN
-F 4 "311-21.0KCRCT-ND" H 10000 3050 50  0001 C CNN "Digikey"
-	1    10000 3050
+P 10200 3050
+F 0 "R622" H 10130 3004 50  0000 R CNN
+F 1 "21k" H 10130 3095 50  0000 R CNN
+F 2 "Resistor_SMD:R_0805_2012Metric" V 10130 3050 50  0001 C CNN
+F 3 "~" H 10200 3050 50  0001 C CNN
+F 4 "311-21.0KCRCT-ND" H 10200 3050 50  0001 C CNN "Digikey"
+	1    10200 3050
 	0    -1   -1   0
 $EndComp
@@
 L power:+5V #PWR0629
 U 1 1 5A82849A
-P 10250 2950
-F 0 "#PWR0629" H 10250 2800 50  0001 C CNN
-F 1 "+5V" H 10265 3123 50  0000 C CNN
-F 2 "" H 10250 2950 50  0001 C CNN
-F 3 "" H 10250 2950 50  0001 C CNN
-	1    10250 2950
-	1    0    0    -1
-$EndComp
-Wire Wire Line
-	10150 3050 10250 3050
-Wire Wire Line
-	10250 3050 10250 2950
-Wire Wire Line
-	9750 3050 9850 3050
-Wire Wire Line
-	9450 3050 9350 3050
-Wire Wire Line
-	8850 1650 8850 3550
-Connection ~ 8950 1650
-Wire Wire Line
-	8950 1650 9250 1650
-Wire Wire Line
-	8950 3050 9050 3050
-Wire Wire Line
-	8950 1650 8950 3050
+P 10450 2950
+F 0 "#PWR0629" H 10450 2800 50  0001 C CNN
+F 1 "+5V" H 10465 3123 50  0000 C CNN
+F 2 "" H 10450 2950 50  0001 C CNN
+F 3 "" H 10450 2950 50  0001 C CNN
+	1    10450 2950
+	1    0    0    -1
+$EndComp
+Wire Wire Line
+	10350 3050 10450 3050
+Wire Wire Line
+	10450 3050 10450 2950
+Wire Wire Line
+	9950 3050 10050 3050
+Wire Wire Line
+	9650 3050 9550 3050
+Wire Wire Line
+	8750 1650 8750 3550
+Connection ~ 8850 1650
+Wire Wire Line
+	8850 1650 9050 1650
+Wire Wire Line
+	8850 1650 8850 3050
 $Comp
 L Device:D_Zener D608
 U 1 1 5A83F6A5
-P 9250 2050
-F 0 "D608" V 9204 2129 50  0000 L CNN
-F 1 "1.5SMC400CA" V 9295 2129 50  0000 L CNN
-F 2 "Diode_SMD:D_SMC" H 9250 2050 50  0001 C CNN
-F 3 "http://www.littelfuse.com/~/media/electronics/datasheets/tvs_diodes/littelfuse_tvs_diode_1_5smc_datasheet.pdf.pdf" H 9250 2050 50  0001 C CNN
-F 4 "1.5SMC400CACT-ND" V 9250 2050 50  0001 C CNN "Digikey"
-F 5 "1.5SMC400CA" V 9250 2050 50  0001 C CNN "Mfg part"
-	1    9250 2050
+P 9050 1900
+F 0 "D608" V 9004 1979 50  0000 L CNN
+F 1 "1.5SMC400CA" V 9095 1979 50  0000 L CNN
+F 2 "Diode_SMD:D_SMC" H 9050 1900 50  0001 C CNN
+F 3 "http://www.littelfuse.com/~/media/electronics/datasheets/tvs_diodes/littelfuse_tvs_diode_1_5smc_datasheet.pdf.pdf" H 9050 1900 50  0001 C CNN
+F 4 "1.5SMC400CACT-ND" V 9050 1900 50  0001 C CNN "Digikey"
+F 5 "1.5SMC400CA" V 9050 1900 50  0001 C CNN "Mfg part"
+	1    9050 1900
 	0    1    1    0
 $EndComp
 Wire Wire Line
-	9250 1900 9250 1650
-Connection ~ 9250 1650
-Wire Wire Line
-	9250 1650 10000 1650
+	9050 1750 9050 1650
 $Comp
 L power:GNDPWR #PWR0630
 U 1 1 5A8670B7
-P 9250 2400
-F 0 "#PWR0630" H 9250 2200 50  0001 C CNN
-F 1 "GNDPWR" H 9250 2200 50  0000 C CNN
-F 2 "" H 9250 2350 50  0001 C CNN
-F 3 "" H 9250 2350 50  0001 C CNN
-	1    9250 2400
-	1    0    0    -1
-$EndComp
-Wire Wire Line
-	9250 2400 9250 2200
+P 9050 2150
+F 0 "#PWR0630" H 9050 1950 50  0001 C CNN
+F 1 "GNDPWR" H 9050 1950 50  0000 C CNN
+F 2 "" H 9050 2100 50  0001 C CNN
+F 3 "" H 9050 2100 50  0001 C CNN
+	1    9050 2150
+	1    0    0    -1
+$EndComp
+Wire Wire Line
+	9050 2150 9050 2050
 $Comp
 L Device:C C615
@@
 L Device:R R623
 U 1 1 5A860AAE
-P 10000 2050
-F 0 "R623" H 9930 2004 50  0000 R CNN
-F 1 "21k" H 9930 2095 50  0000 R CNN
-F 2 "Resistor_SMD:R_0805_2012Metric" V 9930 2050 50  0001 C CNN
-F 3 "~" H 10000 2050 50  0001 C CNN
-F 4 "311-21.0KCRCT-ND" H 10000 2050 50  0001 C CNN "Digikey"
-	1    10000 2050
-	-1   0    0    1
-$EndComp
-Wire Wire Line
-	10000 1900 10000 1650
-Connection ~ 10000 1650
-Wire Wire Line
-	10000 1650 10250 1650
+P 9850 1900
+F 0 "R623" H 9780 1854 50  0000 R CNN
+F 1 "187k" H 9780 1945 50  0000 R CNN
+F 2 "Resistor_SMD:R_0805_2012Metric" V 9780 1900 50  0001 C CNN
+F 3 "~" H 9850 1900 50  0001 C CNN
+F 4 "311-187KCRCT-ND" H 9850 1900 50  0001 C CNN "Digikey"
+	1    9850 1900
+	-1   0    0    1
+$EndComp
+Wire Wire Line
+	9850 1750 9850 1650
 $Comp
 L power:GNDPWR #PWR0631
 U 1 1 5A895063
-P 10000 2400
-F 0 "#PWR0631" H 10000 2200 50  0001 C CNN
-F 1 "GNDPWR" H 10000 2200 50  0000 C CNN
-F 2 "" H 10000 2350 50  0001 C CNN
-F 3 "" H 10000 2350 50  0001 C CNN
-	1    10000 2400
-	1    0    0    -1
-$EndComp
-Wire Wire Line
-	10000 2400 10000 2200
+P 9850 2550
+F 0 "#PWR0631" H 9850 2350 50  0001 C CNN
+F 1 "GNDPWR" H 9850 2350 50  0000 C CNN
+F 2 "" H 9850 2500 50  0001 C CNN
+F 3 "" H 9850 2500 50  0001 C CNN
+	1    9850 2550
+	1    0    0    -1
+$EndComp
+Wire Wire Line
+	9850 2550 9850 2450
+Connection ~ 9050 1650
+Wire Wire Line
+	9050 1650 9850 1650
+Connection ~ 9850 1650
+Wire Wire Line
+	9850 1650 10250 1650
+$Comp
+L Device:R R624
+U 1 1 5A927EE8
+P 9850 2300
+F 0 "R624" H 9780 2254 50  0000 R CNN
+F 1 "187k" H 9780 2345 50  0000 R CNN
+F 2 "Resistor_SMD:R_0805_2012Metric" V 9780 2300 50  0001 C CNN
+F 3 "~" H 9850 2300 50  0001 C CNN
+F 4 "311-187KCRCT-ND" H 9850 2300 50  0001 C CNN "Digikey"
+	1    9850 2300
+	-1   0    0    1
+$EndComp
+Wire Wire Line
+	9850 2150 9850 2050
+Wire Wire Line
+	8850 3050 9250 3050
 $EndSCHEMATC

Commit message: Add BOM
Parts:
- U603, U604: value FAN7371 -> FAN7171; Digikey FAN7371MXDKR-ND -> FAN7171MX-F085FSCT-ND; Mouser 512-FAN7371MX -> (none)
Changed lines of the file:
@@
 P 3600 2850
 F 0 "U603" H 3700 3300 50  0000 C CNN
-F 1 "FAN7371" H 3800 3200 50  0000 C CNN
+F 1 "FAN7171" H 3800 3200 50  0000 C CNN
 F 2 "Package_SO:SOIC-8_3.9x4.9mm_P1.27mm" H 3650 2500 50  0001 L CNN
-F 3 "https://www.fairchildsemi.com/datasheets/FA/FAN7371.pdf" H 3600 2750 50  0001 C CNN
-F 4 "512-FAN7371MX" H 3600 2850 50  0001 C CNN "Mouser"
-F 5 "FAN7371MXDKR-ND" H 3600 2850 50  0001 C CNN "Digikey"
+F 3 "https://www.fairchildsemi.com/datasheets/FA/FAN7171_F085.pdf" H 3600 2750 50  0001 C CNN
+F 4 "FAN7171MX-F085FSCT-ND" H 3600 2850 50  0001 C CNN "Digikey"
 	1    3600 2850
 	1    0    0    -1
@@
 Wire Wire Line
 	6350 5750 8850 5750
-$Comp
-L Driver_FET:FAN7371 U604
-U 1 1 5A83AD77
-P 5900 2850
-F 0 "U604" H 6000 3300 50  0000 C CNN
-F 1 "FAN7371" H 6100 3200 50  0000 C CNN
-F 2 "Package_SO:SOIC-8_3.9x4.9mm_P1.27mm" H 5950 2500 50  0001 L CNN
-F 3 "https://www.fairchildsemi.com/datasheets/FA/FAN7371.pdf" H 5900 2750 50  0001 C CNN
-F 4 "512-FAN7371MX" H 5900 2850 50  0001 C CNN "Mouser"
-F 5 "FAN7371MXDKR-ND" H 5900 2850 50  0001 C CNN "Digikey"
-	1    5900 2850
-	1    0    0    -1
-$EndComp
 $Comp
 L power:GNDPWR #PWR0624
@@
 Wire Wire Line
 	8850 3050 9250 3050
+$Comp
+L Driver_FET:FAN7371 U604
+U 1 1 5A8D9CBA
+P 5900 2850
+F 0 "U604" H 6000 3300 50  0000 C CNN
+F 1 "FAN7171" H 6100 3200 50  0000 C CNN
+F 2 "Package_SO:SOIC-8_3.9x4.9mm_P1.27mm" H 5950 2500 50  0001 L CNN
+F 3 "https://www.fairchildsemi.com/datasheets/FA/FAN7171_F085.pdf" H 5900 2750 50  0001 C CNN
+F 4 "FAN7171MX-F085FSCT-ND" H 5900 2850 50  0001 C CNN "Digikey"
+	1    5900 2850
+	1    0    0    -1
+$EndComp
 $EndSCHEMATC
