File: hardware/edm_control_board/cad/edm_control_board/power_management.sch (KiCad schematic (older format))
At the start: 0 parts

Commit message: Power supply
Parts:
- added C301, C302: 330n, Capacitor_SMD:C_0805_2012Metric, symbol Device:C
- added C303, C304: 100n, Capacitor_SMD:C_0805_2012Metric, symbol Device:C
- added C305, C306: 10u, Capacitor_SMD:CP_Elec_6.3x5.3, symbol Device:C
- added NT301: Net-Tie_2, NetTie:NetTie-2_SMD_Pad2.0mm, symbol Device:Net-Tie_2
- added U302: R-78E3.3-1.0, Converter_DCDC:Converter_DCDC_RECOM_R-78E-0.5_THT, symbol Regulator_Switching:R-78E3.3-1.0
- added U303: L78L05_SO8, Package_SO:SOIC-8_3.9x4.9mm_P1.27mm, symbol Regulator_Linear:L78L05_SO8
Connections:
- net labels added: +24V, +3.3V, +3V3, +5V, GND, GNDPWR
- wire segments 0 -> 44
