File: hardware/edm_control_board/cad/edm_control_board/controller.sch (KiCad schematic (older format))
At the start: 1 part

Commit message: Main sheet
Parts:
- added Q? (x3): BSS214NW, Package_TO_SOT_SMD:SOT-323_SC-70, symbol Transistor_FET:BSS214NW
- added R? (x3): 47k, Resistor_SMD:R_0805_2012Metric, symbol Device:R
- gave numbers to parts that had none: 1
Connections:
- net labels added: GND, Stepper_DIR, Stepper_EN, Stepper_PUL
- wire segments 0 -> 27
Changed lines of the file:
@@
 $EndDescr
 $Comp
-L MCU_ST_STM32F7:STM32F722RETx U?
+L MCU_ST_STM32F7:STM32F722RETx U301
 U 1 1 5A8A1ADB
 P 3300 3900
-F 0 "U?" H 3250 5878 50  0000 C CNN
+F 0 "U301" H 3250 5878 50  0000 C CNN
 F 1 "STM32F722RETx" H 3250 5787 50  0000 C CNN
 F 2 "Package_QFP:LQFP-64_10x10mm_P0.5mm" H 2700 2200 50  0001 R CNN
@@
 	1    0    0    -1
 $EndComp
+$Comp
+L Transistor_FET:BSS214NW Q?
+U 1 1 5A8B3057
+P 9900 1500
+F 0 "Q?" H 10105 1546 50  0000 L CNN
+F 1 "BSS214NW" H 10105 1455 50  0000 L CNN
+F 2 "Package_TO_SOT_SMD:SOT-323_SC-70" H 10100 1425 50  0001 L CIN
+F 3 "https://www.infineon.com/dgdl/Infineon-BSS214NW-DS-v02_02-en.pdf?fileId=db3a30431b3e89eb011b695aebc01bde" H 9900 1500 50  0001 L CNN
+F 4 "BSS214NWH6327XTSA1" H 9900 1500 50  0001 C CNN "Digikey"
+	1    9900 1500
+	1    0    0    -1
+$EndComp
+$Comp
+L power:GND #PWR?
+U 1 1 5A8B30C5
+P 10000 2100
+F 0 "#PWR?" H 10000 1850 50  0001 C CNN
+F 1 "GND" H 10005 1927 50  0000 C CNN
+F 2 "" H 10000 2100 50  0001 C CNN
+F 3 "" H 10000 2100 50  0001 C CNN
+	1    10000 2100
+	1    0    0    -1
+$EndComp
+Wire Wire Line
+	10000 2100 10000 2000
+Text HLabel 10200 1200 2    50   Input ~ 0
+Stepper_PUL
+Wire Wire Line
+	10000 1300 10000 1200
+Wire Wire Line
+	10000 1200 10200 1200
+$Comp
+L Device:R R?
+U 1 1 5A8B3255
+P 9600 1750
+F 0 "R?" H 9670 1796 50  0000 L CNN
+F 1 "47k" H 9670 1705 50  0000 L CNN
+F 2 "Resistor_SMD:R_0805_2012Metric" V 9530 1750 50  0001 C CNN
+F 3 "~" H 9600 1750 50  0001 C CNN
+F 4 "311-27.0KCRCT-ND" H 9600 1750 50  0001 C CNN "Digikey"
+	1    9600 1750
+	1    0    0    -1
+$EndComp
+Wire Wire Line
+	9600 1900 9600 2000
+Wire Wire Line
+	9600 2000 10000 2000
+Connection ~ 10000 2000
+Wire Wire Line
+	10000 2000 10000 1700
+Wire Wire Line
+	9600 1600 9600 1500
+Wire Wire Line
+	9600 1500 9700 1500
+Wire Wire Line
+	9600 1500 9100 1500
+Connection ~ 9600 1500
+$Comp
+L Transistor_FET:BSS214NW Q?
+U 1 1 5A8D715C
+P 9900 2800
+F 0 "Q?" H 10105 2846 50  0000 L CNN
+F 1 "BSS214NW" H 10105 2755 50  0000 L CNN
+F 2 "Package_TO_SOT_SMD:SOT-323_SC-70" H 10100 2725 50  0001 L CIN
+F 3 "https://www.infineon.com/dgdl/Infineon-BSS214NW-DS-v02_02-en.pdf?fileId=db3a30431b3e89eb011b695aebc01bde" H 9900 2800 50  0001 L CNN
+F 4 "BSS214NWH6327XTSA1" H 9900 2800 50  0001 C CNN "Digikey"
+	1    9900 2800
+	1    0    0    -1
+$EndComp
+$Comp
+L power:GND #PWR?
+U 1 1 5A8D7162
+P 10000 3400
+F 0 "#PWR?" H 10000 3150 50  0001 C CNN
+F 1 "GND" H 10005 3227 50  0000 C CNN
+F 2 "" H 10000 3400 50  0001 C CNN
+F 3 "" H 10000 3400 50  0001 C CNN
+	1    10000 3400
+	1    0    0    -1
+$EndComp
+Wire Wire Line
+	10000 3400 10000 3300
+Text HLabel 10200 2500 2    50   Input ~ 0
+Stepper_DIR
+Wire Wire Line
+	10000 2600 10000 2500
+Wire Wire Line
+	10000 2500 10200 2500
+$Comp
+L Device:R R?
+U 1 1 5A8D716D
+P 9600 3050
+F 0 "R?" H 9670 3096 50  0000 L CNN
+F 1 "47k" H 9670 3005 50  0000 L CNN
+F 2 "Resistor_SMD:R_0805_2012Metric" V 9530 3050 50  0001 C CNN
+F 3 "~" H 9600 3050 50  0001 C CNN
+F 4 "311-27.0KCRCT-ND" H 9600 3050 50  0001 C CNN "Digikey"
+	1    9600 3050
+	1    0    0    -1
+$EndComp
+Wire Wire Line
+	9600 3200 9600 3300
+Wire Wire Line
+	9600 3300 10000 3300
+Connection ~ 10000 3300
+Wire Wire Line
+	10000 3300 10000 3000
+Wire Wire Line
+	9600 2900 9600 2800
+Wire Wire Line
+	9600 2800 9700 2800
+Wire Wire Line
+	9600 2800 9100 2800
+Connection ~ 9600 2800
+$Comp
+L Transistor_FET:BSS214NW Q?
+U 1 1 5A8D80FD
+P 9900 4100
+F 0 "Q?" H 10105 4146 50  0000 L CNN
+F 1 "BSS214NW" H 10105 4055 50  0000 L CNN
+F 2 "Package_TO_SOT_SMD:SOT-323_SC-70" H 10100 4025 50  0001 L CIN
+F 3 "https://www.infineon.com/dgdl/Infineon-BSS214NW-DS-v02_02-en.pdf?fileId=db3a30431b3e89eb011b695aebc01bde" H 9900 4100 50  0001 L CNN
+F 4 "BSS214NWH6327XTSA1" H 9900 4100 50  0001 C CNN "Digikey"
+	1    9900 4100
+	1    0    0    -1
+$EndComp
+$Comp
+L power:GND #PWR?
+U 1 1 5A8D8103
+P 10000 4700
+F 0 "#PWR?" H 10000 4450 50  0001 C CNN
+F 1 "GND" H 10005 4527 50  0000 C CNN
+F 2 "" H 10000 4700 50  0001 C CNN
+F 3 "" H 10000 4700 50  0001 C CNN
+	1    10000 4700
+	1    0    0    -1
+$EndComp
+Wire Wire Line
+	10000 4700 10000 4600
+Text HLabel 10200 3800 2    50   Input ~ 0
+Stepper_EN
+Wire Wire Line
+	10000 3900 10000 3800
+Wire Wire Line
+	10000 3800 10200 3800
+$Comp
+L Device:R R?
+U 1 1 5A8D810E
+P 9600 4350
+F 0 "R?" H 9670 4396 50  0000 L CNN
+F 1 "47k" H 9670 4305 50  0000 L CNN
+F 2 "Resistor_SMD:R_0805_2012Metric" V 9530 4350 50  0001 C CNN
+F 3 "~" H 9600 4350 50  0001 C CNN
+F 4 "311-27.0KCRCT-ND" H 9600 4350 50  0001 C CNN "Digikey"
+	1    9600 4350
+	1    0    0    -1
+$EndComp
+Wire Wire Line
+	9600 4500 9600 4600
+Wire Wire Line
+	9600 4600 10000 4600
+Connection ~ 10000 4600
+Wire Wire Line
+	10000 4600 10000 4300
+Wire Wire Line
+	9600 4200 9600 4100
+Wire Wire Line
+	9600 4100 9700 4100
+Wire Wire Line
+	9600 4100 9100 4100
+Connection ~ 9600 4100
 $EndSCHEMATC

Commit message: Power supply
Parts:
- added C201, C202, C203, C204, C205: 100n, Capacitor_SMD:C_0805_2012Metric, symbol Device:C
- added C206: 1u, Capacitor_SMD:C_0805_2012Metric, symbol Device:C
- added Q201: BSS214NW, Package_TO_SOT_SMD:SOT-323_SC-70, symbol Transistor_FET:BSS214NW
- added R201: 27k, Resistor_SMD:R_0805_2012Metric, symbol Device:R
- added R205: 20R, Resistor_SMD:R_0805_2012Metric, symbol Device:R
- added RV201: 20k, Potentiometer_SMD:Potentiometer_Bourns_3214X_Vertical, symbol Device:POT
- R202, R203, R204: renamed from R?; value 47k -> 27k
- gave numbers to parts that had none: 3
Connections:
- net labels added: +3.3V, +3V3, LCD_A, LCD_DB0, LCD_DB1, LCD_DB2, LCD_DB3, LCD_DB4, LCD_DB5, LCD_DB6, LCD_DB7, LCD_E, LCD_K, LCD_RS, LCD_RW, LCD_V0
- wire segments 27 -> 69

Commit message: Microcontroller
Parts:
- added C206, C209: 100n, Capacitor_SMD:C_0805_2012Metric, symbol Device:C
- added C208, C210: 12p, Capacitor_SMD:C_0805_2012Metric, symbol Device:C
- added C211, C212: 2u2, Capacitor_SMD:C_0805_2012Metric, symbol Device:C
- added R206, R207: 27k, Resistor_SMD:R_0805_2012Metric, symbol Device:R
- added Y201: 25M, Crystal:Crystal_SMD_5032-2Pin_5.0x3.2mm, symbol Device:Crystal_Small
- renumbered C206 to C207
Connections:
- net labels added: Breakdown, Output_20V_Enable, Output_250V_Enable, Short_Circuit, Spark_Voltage_0, Spark_Voltage_1, Spark_Voltage_2, Spark_Voltage_Status
- wire segments 69 -> 150
Other:
- moved on the sheet: U301
