File: hardware/edm_control_board/cad/edm_control_board/edm_control_board.kicad_pcb (KiCad board)
At the start: 2 copper layers, 240 x 100 mm, 26 parts, among them J501 Conn_02x08_Odd_Even, J502 Conn_01x02, SW401 SW_Push, SW402 SW_Push, SW403 SW_Push, SW404 SW_Push, U301 STM32F722RETx, U401 NHD-0420H1Z

Commit message: Power supply
Parts:
- added C201: 100n, Capacitor_SMD:C_0805_2012Metric, B.Cu at (116.2, -126.7)
- added C202: 100n, Capacitor_SMD:C_0805_2012Metric, B.Cu at (124.7, -120.7)
- added C203: 100n, Capacitor_SMD:C_0805_2012Metric, B.Cu at (130.4, -120.4)
- added C204: 100n, Capacitor_SMD:C_0805_2012Metric, B.Cu at (120.6, -126.7)
- added C205: 100n, Capacitor_SMD:C_0805_2012Metric, B.Cu at (134.8, -120.4)
- added C206: 1u, Capacitor_SMD:C_0805_2012Metric, B.Cu at (134.8, -114.6)
- added C301: 330n, Capacitor_SMD:C_0805_2012Metric, B.Cu at (107.7, -150.8)
- added C302: 330n, Capacitor_SMD:C_0805_2012Metric, B.Cu at (116.5, -150.8)
- added C303: 100n, Capacitor_SMD:C_0805_2012Metric, B.Cu at (127.4, -148.7)
- added C304: 100n, Capacitor_SMD:C_0805_2012Metric, B.Cu at (112.1, -150.8)
- added C305: 10u, Capacitor_SMD:CP_Elec_6.3x5.3, B.Cu at (120.2, -142.4)
- added C306: 10u, Capacitor_SMD:CP_Elec_6.3x5.3, B.Cu at (110.4, -142.4)
- added NT301: Net-Tie_2, NetTie:NetTie-2_SMD_Pad2.0mm, B.Cu at (82.7, -132.0)
- added Q201: BSS214NW, Package_TO_SOT_SMD:SOT-323_SC-70, B.Cu at (109.8, -126.3)
- added Q202: BSS214NW, Package_TO_SOT_SMD:SOT-323_SC-70, B.Cu at (115.5, -114.7)
- added Q203: BSS214NW, Package_TO_SOT_SMD:SOT-323_SC-70, B.Cu at (124.0, -114.7)
- added Q204: BSS214NW, Package_TO_SOT_SMD:SOT-323_SC-70, B.Cu at (118.3, -120.8)
- added R201: 27k, Resistor_SMD:R_0805_2012Metric, B.Cu at (129.1, -126.1)
- added R202: 27k, Resistor_SMD:R_0805_2012Metric, B.Cu at (139.2, -114.6)
- added R203: 27k, Resistor_SMD:R_0805_2012Metric, B.Cu at (139.2, -120.4)
- added R204: 27k, Resistor_SMD:R_0805_2012Metric, B.Cu at (133.5, -126.1)
- added R205: 20R, Resistor_SMD:R_0805_2012Metric, B.Cu at (130.4, -114.6)
- added RV201: 20k, Potentiometer_SMD:Potentiometer_Bourns_3214X_Vertical, B.Cu at (108.4, -117.5)
- added U302: R-78E3.3-1.0, Converter_DCDC:Converter_DCDC_RECOM_R-78E-0.5_THT, B.Cu at (69.8, -126.5)
- added U303: L78L05_SO8, Package_SO:SOIC-8_3.9x4.9mm_P1.27mm, B.Cu at (130.0, -141.3)
- moved U301 57.7 mm to (172.0, -47.0)
- moved SW401 5.00 mm to (42.0, -35.0)
- moved SW402 5.00 mm to (82.0, -35.0)
- moved SW403 5.00 mm to (42.0, -20.0)
- moved SW404 5.00 mm to (82.0, -20.0)
Connections:
- J502 pad 1: /Connectors/GNDPWR -> GND
- J502 pad 2: /Connectors/+24V -> +24V
- JJ504 pad 1: /Connectors/Stepper_+5V -> +5V
- MK501 pad 1: /Connectors/GNDPWR -> GND
- MK502 pad 1: /Connectors/GNDPWR -> GND
- MK503 pad 1: /Connectors/GNDPWR -> GND
- MK504 pad 1: /Connectors/GNDPWR -> GND
- MK505 pad 1: /Connectors/GNDPWR -> GND
- MK506 pad 1: /Connectors/GNDPWR -> GND
- MK507 pad 1: /Connectors/GNDPWR -> GND
- MK508 pad 1: /Connectors/GNDPWR -> GND
- MK509 pad 1: /Connectors/GNDPWR -> GND
- MK510 pad 1: /Connectors/GNDPWR -> GND
- MK511 pad 1: /Connectors/GNDPWR -> GND
- MK512 pad 1: /Connectors/GNDPWR -> GND

Commit message: Microcontroller
Parts:
- added C207: 1u, Capacitor_SMD:C_0805_2012Metric, B.Cu at (50.3, -132.0)
- added C208: 12p, Capacitor_SMD:C_0805_2012Metric, B.Cu at (45.9, -137.8)
- added C209: 100n, Capacitor_SMD:C_0805_2012Metric, B.Cu at (50.3, -137.8)
- added C210: 12p, Capacitor_SMD:C_0805_2012Metric, B.Cu at (54.7, -132.0)
- added C211: 2u2, Capacitor_SMD:C_0805_2012Metric, B.Cu at (59.1, -132.0)
- added C212: 2u2, Capacitor_SMD:C_0805_2012Metric, B.Cu at (54.7, -137.8)
- added R206: 27k, Resistor_SMD:R_0805_2012Metric, B.Cu at (45.9, -132.0)
- added R207: 27k, Resistor_SMD:R_0805_2012Metric, B.Cu at (39.2, -139.7)
- added Y201: 25M, Crystal:Crystal_SMD_5032-2Pin_5.0x3.2mm, B.Cu at (40.3, -133.0)
- C206: value 1u -> 100n
Connections:
- net /User Interface/LCD_K renamed /Controller/LCD_K
- net /User Interface/LCD_V0 renamed /Controller/LCD_V0
- C206 pad 1: /User Interface/LCD_A -> +3V3
- R205 pad 1: /User Interface/LCD_A -> /Controller/LCD_A
- U301 pad 1: Net-(U301-Pad1) -> +3V3
- U301 pad 12: Net-(U301-Pad12) -> GND
- U301 pad 13: Net-(U301-Pad13) -> +3V3
- U301 pad 14: Net-(U301-Pad14) -> /Controller/LCD_DB0
- U301 pad 15: Net-(U301-Pad15) -> /Controller/LCD_DB1
- U301 pad 16: Net-(U301-Pad16) -> /Controller/LCD_DB2
- U301 pad 17: Net-(U301-Pad17) -> /Controller/LCD_DB3
- U301 pad 18: Net-(U301-Pad18) -> GND
- U301 pad 19: Net-(U301-Pad19) -> +3V3
- U301 pad 20: Net-(U301-Pad20) -> /Controller/LCD_DB4
- U301 pad 21: Net-(U301-Pad21) -> /Controller/LCD_DB5
- U301 pad 22: Net-(U301-Pad22) -> /Controller/LCD_DB6
- U301 pad 23: Net-(U301-Pad23) -> /Controller/LCD_DB7
- U301 pad 25: Net-(U301-Pad25) -> /Connectors/Spark_Voltage_0
- U301 pad 26: Net-(U301-Pad26) -> /Connectors/Spark_Voltage_1
- U301 pad 27: Net-(U301-Pad27) -> /Connectors/Spark_Voltage_2
- U301 pad 31: Net-(U301-Pad31) -> GND
- U301 pad 32: Net-(U301-Pad32) -> +3V3
- U301 pad 41: Net-(U301-Pad41) -> /Controller/LCD_RS
- U301 pad 42: Net-(U301-Pad42) -> /Controller/LCD_RW
- U301 pad 43: Net-(U301-Pad43) -> /Controller/LCD_E
- U301 pad 45: Net-(U301-Pad45) -> Net-(Q202-Pad1)
- U301 pad 46: Net-(U301-Pad46) -> Net-(Q203-Pad1)
- U301 pad 47: Net-(U301-Pad47) -> GND
- U301 pad 48: Net-(U301-Pad48) -> +3V3
- U301 pad 49: Net-(U301-Pad49) -> Net-(Q204-Pad1)
- U301 pad 50: Net-(U301-Pad50) -> Net-(Q201-Pad1)
- U301 pad 55: Net-(U301-Pad55) -> /Connectors/Spark_Voltage_Status
- U301 pad 56: Net-(U301-Pad56) -> /Connectors/Output_250V_Enable
- U301 pad 57: Net-(U301-Pad57) -> /Connectors/Output_20V_Enable
- U301 pad 58: Net-(U301-Pad58) -> /Connectors/Short_Circuit
- U301 pad 59: Net-(U301-Pad59) -> /Connectors/Breakdown
- U301 pad 63: Net-(U301-Pad63) -> GND
- U301 pad 64: Net-(U301-Pad64) -> +3V3
- U401 pad 10: /User Interface/LCD_DB3 -> /Controller/LCD_DB3
- U401 pad 11: /User Interface/LCD_DB4 -> /Controller/LCD_DB4
- U401 pad 12: /User Interface/LCD_DB5 -> /Controller/LCD_DB5
- U401 pad 13: /User Interface/LCD_DB6 -> /Controller/LCD_DB6
- U401 pad 14: /User Interface/LCD_DB7 -> /Controller/LCD_DB7
- U401 pad 15: /User Interface/LCD_A -> /Controller/LCD_A
- U401 pad 4: /User Interface/LCD_RS -> /Controller/LCD_RS
- U401 pad 5: /User Interface/LCD_RW -> /Controller/LCD_RW
- U401 pad 6: /User Interface/LCD_E -> /Controller/LCD_E
- U401 pad 7: /User Interface/LCD_DB0 -> /Controller/LCD_DB0
- U401 pad 8: /User Interface/LCD_DB1 -> /Controller/LCD_DB1
- U401 pad 9: /User Interface/LCD_DB2 -> /Controller/LCD_DB2
