File: hardware/edm_control_board/cad/edm_control_board/edm_control_board.sch (KiCad schematic (older format))
At the start: 0 parts

Commit message: Main sheet
Connections:
- net labels added: +24V, +3.3V, +5V, GND, GNDPWR
- wire segments 54 -> 57

Commit message: Microcontroller
Changed lines of the file:
@@
 S 1800 1900 950  4250
 U 5A95285C
-F0 "controller" 50
+F0 "Controller" 50
 F1 "controller.sch" 50
 F2 "+3V3" I L 1800 2000 50
@@
 S 8000 3450 1200 400
 U 5A89896C
-F0 "power_management" 50
+F0 "Power Management" 50
 F1 "power_management.sch" 50
 F2 "+24V" I L 8000 3550 50
