File: hardware/edm_control_board/cad/edm_control_board.sch (KiCad schematic (older format))
At the start: 0 parts

Commit message: Component placement
Changed lines of the file:
@@
 $EndSheet
-Wire Wire Line
-	5500 2000 5700 2000
-Wire Wire Line
-	5700 2100 5500 2100
 Wire Wire Line
 	2750 4950 4550 4950
@@
 Wire Wire Line
 	4550 4300 2750 4300
+Wire Wire Line
+	5550 2000 5700 2000
+Wire Wire Line
+	5700 2100 5550 2100
 $EndSCHEMATC

Commit message: Add SWD connector
Connections:
- wire segments 57 -> 64
Changed lines of the file:
@@
 $EndDescr
 $Sheet
-S 1800 1900 950  4250
+S 1800 1900 950  4650
 U 5A95285C
 F0 "Controller" 50
@@
 F35 "Short_Circuit" I R 2750 5950 50
 F36 "Breakdown" I R 2750 6050 50
+F37 "SWDIO" I R 2750 6250 50
+F38 "SWCLK" I R 2750 6350 50
+F39 "SWO" I R 2750 6450 50
 $EndSheet
 $Sheet
@@
 	4400 4850 4550 4850
 $Sheet
-S 4550 4750 1000 1400
+S 4550 4750 1000 1800
 U 5A952859
 F0 "Connectors" 50
@@
 F14 "Stepper_EN" I L 4550 5150 50
 F15 "Stepper_+5V" I L 4550 4850 50
+F16 "SWDIO" I L 4550 6250 50
+F17 "SWCLK" I L 4550 6350 50
+F18 "SWO" I L 4550 6450 50
+F19 "GND" I R 5550 6450 50
+F20 "+3V3" I R 5550 6350 50
 $EndSheet
 $Sheet
@@
 Wire Wire Line
 	5700 2100 5550 2100
+Wire Wire Line
+	2750 6250 4550 6250
+Wire Wire Line
+	4550 6350 2750 6350
+Wire Wire Line
+	2750 6450 4550 6450
+$Comp
+L power:GND #PWR062
+U 1 1 5A9A893F
+P 5700 6550
+F 0 "#PWR062" H 5700 6300 50  0001 C CNN
+F 1 "GND" H 5705 6377 50  0000 C CNN
+F 2 "" H 5700 6550 50  0001 C CNN
+F 3 "" H 5700 6550 50  0001 C CNN
+	1    5700 6550
+	1    0    0    -1
+$EndComp
+Wire Wire Line
+	5700 6550 5700 6450
+Wire Wire Line
+	5700 6450 5550 6450
+$Comp
+L power:+3.3V #PWR?
+U 1 1 5A89F810
+P 5700 6250
+F 0 "#PWR?" H 5700 6100 50  0001 C CNN
+F 1 "+3.3V" H 5715 6423 50  0000 C CNN
+F 2 "" H 5700 6250 50  0001 C CNN
+F 3 "" H 5700 6250 50  0001 C CNN
+	1    5700 6250
+	1    0    0    -1
+$EndComp
+Wire Wire Line
+	5700 6250 5700 6350
+Wire Wire Line
+	5550 6350 5700 6350
 $EndSCHEMATC

Commit message: Add water pump output
Connections:
- wire segments 64 -> 93
