File: hardware/edm_control_board/cad/power_management.sch (KiCad schematic (older format))
At the start: 9 parts, among them U302 R-78E3.3-1.0, U303 L78L05_SO8

Commit message: Add water pump output
Parts:
- removed C305, C306: 10u, Capacitor_SMD:CP_Elec_6.3x5.3, symbol Device:C
- added C305, C306: 10u, Capacitor_SMD:CP_Elec_6.3x5.3, symbol Device:CP
Changed lines of the file:
@@
 $Descr A4 11693 8268
 encoding utf-8
-Sheet 3 5
+Sheet 3 6
 Title ""
 Date ""
@@
 	1    0    0    -1
 $EndComp
-$Comp
-L Device:C C305
-U 1 1 5A9CB1D0
-P 6700 2750
-F 0 "C305" H 6815 2796 50  0000 L CNN
-F 1 "10u" H 6815 2705 50  0000 L CNN
-F 2 "Capacitor_SMD:CP_Elec_6.3x5.3" H 6738 2600 50  0001 C CNN
-F 3 "~" H 6700 2750 50  0001 C CNN
-F 4 "PCE4209CT-ND" H 6700 2750 50  0001 C CNN "Digikey"
-	1    6700 2750
-	1    0    0    -1
-$EndComp
 Wire Wire Line
 	6700 2900 6700 3100
@@
 	1    0    0    -1
 $EndComp
-$Comp
-L Device:C C306
-U 1 1 5A9D144B
-P 6700 4400
-F 0 "C306" H 6815 4446 50  0000 L CNN
-F 1 "10u" H 6815 4355 50  0000 L CNN
-F 2 "Capacitor_SMD:CP_Elec_6.3x5.3" H 6738 4250 50  0001 C CNN
-F 3 "~" H 6700 4400 50  0001 C CNN
-F 4 "PCE4209CT-ND" H 6700 4400 50  0001 C CNN "Digikey"
-	1    6700 4400
-	1    0    0    -1
-$EndComp
 Wire Wire Line
 	6700 4550 6700 4750
@@
 	1    0    0    -1
 $EndComp
+$Comp
+L Device:CP C305
+U 1 1 5A8E59FE
+P 6700 2750
+F 0 "C305" H 6818 2796 50  0000 L CNN
+F 1 "10u" H 6818 2705 50  0000 L CNN
+F 2 "Capacitor_SMD:CP_Elec_6.3x5.3" H 6738 2600 50  0001 C CNN
+F 3 "PCE4209CT-ND" H 6700 2750 50  0001 C CNN
+	1    6700 2750
+	1    0    0    -1
+$EndComp
+$Comp
+L Device:CP C306
+U 1 1 5A8E5B90
+P 6700 4400
+F 0 "C306" H 6818 4446 50  0000 L CNN
+F 1 "10u" H 6818 4355 50  0000 L CNN
+F 2 "Capacitor_SMD:CP_Elec_6.3x5.3" H 6738 4250 50  0001 C CNN
+F 3 "PCE4209CT-ND" H 6700 4400 50  0001 C CNN
+	1    6700 4400
+	1    0    0    -1
+$EndComp
