File: hardware/edm_control_board/cad/controller.sch (KiCad schematic (older format))
At the start: 26 parts, among them Q201 BSS214NW, Q202 BSS214NW, Q203 BSS214NW, Q204 BSS214NW, U301 STM32F722RETx, Y201 25M

Commit message: Change to horizontal trim pot
Parts:
- RV201: footprint Potentiometer_SMD:Potentiometer_Bourns_3214X_Vertical -> Potentiometer_SMD:Potentiometer_Bourns_3214J_Horizontal; Digikey 3214X-1-203ECT-ND -> 3214J-203ECT-ND
Changed lines of the file:
@@
 F 0 "RV201" H 1381 6996 50  0000 R CNN
 F 1 "20k" H 1381 6905 50  0000 R CNN
-F 2 "Potentiometer_SMD:Potentiometer_Bourns_3214X_Vertical" H 1450 6950 50  0001 C CNN
+F 2 "Potentiometer_SMD:Potentiometer_Bourns_3214J_Horizontal" H 1450 6950 50  0001 C CNN
 F 3 "http://www.bourns.com/docs/Product-Datasheets/3214.pdf" H 1450 6950 50  0001 C CNN
-F 4 "3214X-1-203ECT-ND" H 1450 6950 50  0001 C CNN "Digikey"
+F 4 "3214J-203ECT-ND" H 1450 6950 50  0001 C CNN "Digikey"
 	1    1450 6950
 	-1   0    0    -1

Commit message: Update pinout
Connections:
- wire segments 150 -> 152
Changed lines of the file:
@@
 L Transistor_FET:BSS214NW Q201
 U 1 1 5A97BBD5
-P 8550 5400
-F 0 "Q201" H 8755 5446 50  0000 L CNN
-F 1 "BSS214NW" H 8755 5355 50  0000 L CNN
-F 2 "Package_TO_SOT_SMD:SOT-323_SC-70" H 8750 5325 50  0001 L CIN
-F 3 "https://www.infineon.com/dgdl/Infineon-BSS214NW-DS-v02_02-en.pdf?fileId=db3a30431b3e89eb011b695aebc01bde" H 8550 5400 50  0001 L CNN
-F 4 "BSS214NWH6327XTSA1" H 8550 5400 50  0001 C CNN "Digikey"
-	1    8550 5400
+P 8350 5200
+F 0 "Q201" H 8555 5246 50  0000 L CNN
+F 1 "BSS214NW" H 8555 5155 50  0000 L CNN
+F 2 "Package_TO_SOT_SMD:SOT-323_SC-70" H 8550 5125 50  0001 L CIN
+F 3 "https://www.infineon.com/dgdl/Infineon-BSS214NW-DS-v02_02-en.pdf?fileId=db3a30431b3e89eb011b695aebc01bde" H 8350 5200 50  0001 L CNN
+F 4 "BSS214NWH6327XTSA1" H 8350 5200 50  0001 C CNN "Digikey"
+	1    8350 5200
 	1    0    0    -1
 $EndComp
@@
 L power:GND #PWR032
 U 1 1 5A97BBDB
-P 8650 6000
-F 0 "#PWR032" H 8650 5750 50  0001 C CNN
-F 1 "GND" H 8655 5827 50  0000 C CNN
-F 2 "" H 8650 6000 50  0001 C CNN
-F 3 "" H 8650 6000 50  0001 C CNN
-	1    8650 6000
-	1    0    0    -1
-$EndComp
-Wire Wire Line
-	8650 6000 8650 5900
-Text HLabel 8850 5100 2    50   Input ~ 0
+P 8450 5800
+F 0 "#PWR032" H 8450 5550 50  0001 C CNN
+F 1 "GND" H 8455 5627 50  0000 C CNN
+F 2 "" H 8450 5800 50  0001 C CNN
+F 3 "" H 8450 5800 50  0001 C CNN
+	1    8450 5800
+	1    0    0    -1
+$EndComp
+Wire Wire Line
+	8450 5800 8450 5700
+Text HLabel 8650 4900 2    50   Input ~ 0
 LCD_K
 Wire Wire Line
-	8650 5200 8650 5100
-Wire Wire Line
-	8650 5100 8850 5100
+	8450 5000 8450 4900
+Wire Wire Line
+	8450 4900 8650 4900
 $Comp
 L Device:R R201
 U 1 1 5A97BBE6
-P 8250 5650
-F 0 "R201" H 8320 5696 50  0000 L CNN
-F 1 "27k" H 8320 5605 50  0000 L CNN
-F 2 "Resistor_SMD:R_0805_2012Metric" V 8180 5650 50  0001 C CNN
-F 3 "~" H 8250 5650 50  0001 C CNN
-F 4 "311-27.0KCRCT-ND" H 8250 5650 50  0001 C CNN "Digikey"
-	1    8250 5650
-	1    0    0    -1
-$EndComp
-Wire Wire Line
-	8250 5800 8250 5900
-Wire Wire Line
-	8250 5900 8650 5900
-Connection ~ 8650 5900
-Wire Wire Line
-	8650 5900 8650 5600
-Wire Wire Line
-	8250 5500 8250 5400
-Wire Wire Line
-	8250 5400 8350 5400
-Wire Wire Line
-	8250 5400 7750 5400
-Connection ~ 8250 5400
+P 8050 5450
+F 0 "R201" H 8120 5496 50  0000 L CNN
+F 1 "27k" H 8120 5405 50  0000 L CNN
+F 2 "Resistor_SMD:R_0805_2012Metric" V 7980 5450 50  0001 C CNN
+F 3 "~" H 8050 5450 50  0001 C CNN
+F 4 "311-27.0KCRCT-ND" H 8050 5450 50  0001 C CNN "Digikey"
+	1    8050 5450
+	1    0    0    -1
+$EndComp
+Wire Wire Line
+	8050 5600 8050 5700
+Wire Wire Line
+	8050 5700 8450 5700
+Connection ~ 8450 5700
+Wire Wire Line
+	8450 5700 8450 5400
+Wire Wire Line
+	8050 5300 8050 5200
+Wire Wire Line
+	8050 5200 8150 5200
 Text HLabel 10050 5500 2    50   Input ~ 0
 LCD_A
@@
 Wire Wire Line
 	9450 5500 9550 5500
-Text HLabel 5950 2800 2    50   Input ~ 0
+Text HLabel 5950 3300 2    50   Input ~ 0
 LCD_RS
+Text HLabel 5950 3200 2    50   Input ~ 0
+LCD_RW
+Text HLabel 5950 3100 2    50   Input ~ 0
+LCD_E
+Text HLabel 5950 3000 2    50   Input ~ 0
+LCD_DB0
 Text HLabel 5950 2900 2    50   Input ~ 0
-LCD_RW
-Text HLabel 5950 3000 2    50   Input ~ 0
-LCD_E
-Text HLabel 5950 2000 2    50   Input ~ 0
-LCD_DB0
-Text HLabel 5950 2100 2    50   Input ~ 0
 LCD_DB1
-Text HLabel 5950 2200 2    50   Input ~ 0
+Text HLabel 5950 4400 2    50   Input ~ 0
 LCD_DB2
-Text HLabel 5950 2300 2    50   Input ~ 0
+Text HLabel 5950 4300 2    50   Input ~ 0
 LCD_DB3
-Text HLabel 5950 2400 2    50   Input ~ 0
+Text HLabel 5950 4200 2    50   Input ~ 0
 LCD_DB4
-Text HLabel 5950 2500 2    50   Input ~ 0
+Text HLabel 5950 4100 2    50   Input ~ 0
 LCD_DB5
-Text HLabel 5950 2600 2    50   Input ~ 0
+Text HLabel 5950 4000 2    50   Input ~ 0
 LCD_DB6
-Text HLabel 5950 2700 2    50   Input ~ 0
+Text HLabel 4050 4900 0    50   Input ~ 0
 LCD_DB7
 $Comp
@@
 Wire Wire Line
 	2700 3300 4350 3300
+Text HLabel 5950 4700 2    50   Input ~ 0
+Spark_Voltage_0
+Text HLabel 5950 3900 2    50   Input ~ 0
+Spark_Voltage_1
+Text HLabel 5950 3800 2    50   Input ~ 0
+Spark_Voltage_2
 Text HLabel 5950 3700 2    50   Input ~ 0
-Spark_Voltage_0
-Text HLabel 5950 3800 2    50   Input ~ 0
-Spark_Voltage_1
-Text HLabel 5950 3900 2    50   Input ~ 0
-Spark_Voltage_2
-Text HLabel 5950 4000 2    50   Input ~ 0
 Spark_Voltage_Status
-Text HLabel 5950 4100 2    50   Input ~ 0
+Text HLabel 5950 2700 2    50   Input ~ 0
 Output_250V_Enable
-Text HLabel 5950 4200 2    50   Input ~ 0
+Text HLabel 5950 2600 2    50   Input ~ 0
 Output_20V_Enable
-Text HLabel 5950 4300 2    50   Input ~ 0
+Text HLabel 5950 2500 2    50   Input ~ 0
 Short_Circuit
-Text HLabel 5950 4400 2    50   Input ~ 0
+Text HLabel 5950 2400 2    50   Input ~ 0
 Breakdown
 $Comp
@@
 Connection ~ 2750 2000
 Wire Wire Line
-	7750 5400 7750 3500
-Wire Wire Line
-	7750 3500 5650 3500
-Wire Wire Line
-	5650 3400 7850 3400
-Wire Wire Line
-	7850 3400 7850 4100
-Wire Wire Line
-	7850 4100 9250 4100
-Wire Wire Line
-	5650 3300 7850 3300
-Wire Wire Line
-	7850 3300 7850 2800
-Wire Wire Line
-	7850 2800 9250 2800
-Wire Wire Line
-	5650 3200 7750 3200
-Wire Wire Line
-	7750 3200 7750 1500
-Wire Wire Line
-	7750 1500 9250 1500
-Wire Wire Line
-	5650 2000 5950 2000
-Wire Wire Line
-	5950 2100 5650 2100
-Wire Wire Line
-	5650 2200 5950 2200
-Wire Wire Line
-	5950 2300 5650 2300
+	8950 4000 8950 2800
+Wire Wire Line
+	8950 2800 9250 2800
+Wire Wire Line
+	5650 3000 5950 3000
+Wire Wire Line
+	5950 2900 5650 2900
+Wire Wire Line
+	5650 4400 5950 4400
+Wire Wire Line
+	5950 4300 5650 4300
+Wire Wire Line
+	5650 4200 5950 4200
+Wire Wire Line
+	5950 4100 5650 4100
+Wire Wire Line
+	5650 4000 5950 4000
+Wire Wire Line
+	4050 4900 4350 4900
+Wire Wire Line
+	5650 3300 5950 3300
+Wire Wire Line
+	5950 3200 5650 3200
+Wire Wire Line
+	5650 3100 5950 3100
+Wire Wire Line
+	5950 4700 5650 4700
+Wire Wire Line
+	5650 3900 5950 3900
+Wire Wire Line
+	5950 3800 5650 3800
+Wire Wire Line
+	5650 3700 5950 3700
+Wire Wire Line
+	5950 2700 5650 2700
+Wire Wire Line
+	5650 2600 5950 2600
+Wire Wire Line
+	5950 2500 5650 2500
 Wire Wire Line
 	5650 2400 5950 2400
 Wire Wire Line
-	5950 2500 5650 2500
-Wire Wire Line
-	5650 2600 5950 2600
-Wire Wire Line
-	5950 2700 5650 2700
-Wire Wire Line
-	5650 2800 5950 2800
-Wire Wire Line
-	5950 2900 5650 2900
-Wire Wire Line
-	5650 3000 5950 3000
-Wire Wire Line
-	5950 3700 5650 3700
-Wire Wire Line
-	5650 3800 5950 3800
-Wire Wire Line
-	5950 3900 5650 3900
-Wire Wire Line
-	5650 4000 5950 4000
-Wire Wire Line
-	5950 4100 5650 4100
-Wire Wire Line
-	5650 4200 5950 4200
-Wire Wire Line
-	5950 4300 5650 4300
-Wire Wire Line
-	5650 4400 5950 4400
+	5650 4900 7500 4900
+Wire Wire Line
+	7500 4900 7500 4100
+Wire Wire Line
+	7500 4100 9250 4100
+Wire Wire Line
+	5650 5000 7600 5000
+Wire Wire Line
+	7600 5000 7600 4000
+Wire Wire Line
+	7600 4000 8950 4000
+Wire Wire Line
+	5650 5100 7700 5100
+Wire Wire Line
+	7700 5100 7700 3900
+Wire Wire Line
+	7700 3900 8850 3900
+Wire Wire Line
+	8850 3900 8850 1500
+Wire Wire Line
+	8850 1500 9250 1500
+Wire Wire Line
+	5650 5200 8050 5200
+Connection ~ 8050 5200
 $EndSCHEMATC

Commit message: Update pinout
Connections:
- net labels added: POT_1, POT_2, POT_3, POT_4, SW_1, SW_2, SW_3, SW_4
- wire segments 152 -> 156
Other:
- moved on the sheet: U301

Commit message: Add SWD connector
Connections:
- net labels added: SWCLK, SWDIO, SWO
- wire segments 156 -> 159
Changed lines of the file:
@@
 L Transistor_FET:BSS214NW Q201
 U 1 1 5A97BBD5
-P 7650 3600
-F 0 "Q201" H 7855 3646 50  0000 L CNN
-F 1 "BSS214NW" H 7855 3555 50  0000 L CNN
-F 2 "Package_TO_SOT_SMD:SOT-323_SC-70" H 7850 3525 50  0001 L CIN
-F 3 "https://www.infineon.com/dgdl/Infineon-BSS214NW-DS-v02_02-en.pdf?fileId=db3a30431b3e89eb011b695aebc01bde" H 7650 3600 50  0001 L CNN
-F 4 "BSS214NWH6327XTSA1" H 7650 3600 50  0001 C CNN "Digikey"
-	1    7650 3600
+P 7650 3500
+F 0 "Q201" H 7855 3546 50  0000 L CNN
+F 1 "BSS214NW" H 7855 3455 50  0000 L CNN
+F 2 "Package_TO_SOT_SMD:SOT-323_SC-70" H 7850 3425 50  0001 L CIN
+F 3 "https://www.infineon.com/dgdl/Infineon-BSS214NW-DS-v02_02-en.pdf?fileId=db3a30431b3e89eb011b695aebc01bde" H 7650 3500 50  0001 L CNN
+F 4 "BSS214NWH6327XTSA1" H 7650 3500 50  0001 C CNN "Digikey"
+	1    7650 3500
 	1    0    0    -1
 $EndComp
@@
 L power:GND #PWR032
 U 1 1 5A97BBDB
-P 7750 4200
-F 0 "#PWR032" H 7750 3950 50  0001 C CNN
-F 1 "GND" H 7755 4027 50  0000 C CNN
-F 2 "" H 7750 4200 50  0001 C CNN
-F 3 "" H 7750 4200 50  0001 C CNN
-	1    7750 4200
-	1    0    0    -1
-$EndComp
-Wire Wire Line
-	7750 4200 7750 4100
-Text HLabel 7950 3300 2    50   Input ~ 0
+P 7750 4100
+F 0 "#PWR032" H 7750 3850 50  0001 C CNN
+F 1 "GND" H 7755 3927 50  0000 C CNN
+F 2 "" H 7750 4100 50  0001 C CNN
+F 3 "" H 7750 4100 50  0001 C CNN
+	1    7750 4100
+	1    0    0    -1
+$EndComp
+Wire Wire Line
+	7750 4100 7750 4000
+Text HLabel 7950 3200 2    50   Input ~ 0
 LCD_K
 Wire Wire Line
-	7750 3400 7750 3300
-Wire Wire Line
-	7750 3300 7950 3300
+	7750 3300 7750 3200
+Wire Wire Line
+	7750 3200 7950 3200
 $Comp
 L Device:R R201
 U 1 1 5A97BBE6
-P 7350 3850
-F 0 "R201" H 7420 3896 50  0000 L CNN
-F 1 "27k" H 7420 3805 50  0000 L CNN
-F 2 "Resistor_SMD:R_0805_2012Metric" V 7280 3850 50  0001 C CNN
-F 3 "~" H 7350 3850 50  0001 C CNN
-F 4 "311-27.0KCRCT-ND" H 7350 3850 50  0001 C CNN "Digikey"
-	1    7350 3850
-	1    0    0    -1
-$EndComp
-Wire Wire Line
-	7350 4000 7350 4100
-Wire Wire Line
-	7350 4100 7750 4100
-Connection ~ 7750 4100
-Wire Wire Line
-	7750 4100 7750 3800
-Wire Wire Line
-	7350 3700 7350 3600
-Wire Wire Line
-	7350 3600 7450 3600
+P 7350 3750
+F 0 "R201" H 7420 3796 50  0000 L CNN
+F 1 "27k" H 7420 3705 50  0000 L CNN
+F 2 "Resistor_SMD:R_0805_2012Metric" V 7280 3750 50  0001 C CNN
+F 3 "~" H 7350 3750 50  0001 C CNN
+F 4 "311-27.0KCRCT-ND" H 7350 3750 50  0001 C CNN "Digikey"
+	1    7350 3750
+	1    0    0    -1
+$EndComp
+Wire Wire Line
+	7350 3900 7350 4000
+Wire Wire Line
+	7350 4000 7750 4000
+Connection ~ 7750 4000
+Wire Wire Line
+	7750 4000 7750 3700
+Wire Wire Line
+	7350 3600 7350 3500
+Wire Wire Line
+	7350 3500 7450 3500
 Text HLabel 7850 2250 2    50   Input ~ 0
 LCD_A
@@
 Wire Wire Line
 	7250 2250 7350 2250
-Text HLabel 5900 3500 2    50   Input ~ 0
+Text HLabel 5900 3400 2    50   Input ~ 0
 LCD_RS
-Text HLabel 5900 3400 2    50   Input ~ 0
+Text HLabel 5900 3300 2    50   Input ~ 0
 LCD_RW
-Text HLabel 5900 3300 2    50   Input ~ 0
+Text HLabel 5900 3200 2    50   Input ~ 0
 LCD_E
-Text HLabel 5900 3200 2    50   Input ~ 0
+Text HLabel 5900 3100 2    50   Input ~ 0
 LCD_DB0
-Text HLabel 5900 3100 2    50   Input ~ 0
+Text HLabel 4000 4900 0    50   Input ~ 0
 LCD_DB1
+Text HLabel 5900 4400 2    50   Input ~ 0
+LCD_DB3
 Text HLabel 4000 5200 0    50   Input ~ 0
-LCD_DB3
+LCD_DB4
 Text HLabel 4000 5100 0    50   Input ~ 0
-LCD_DB4
+LCD_DB5
 Text HLabel 4000 5000 0    50   Input ~ 0
-LCD_DB5
+LCD_DB6
+Text HLabel 5900 4500 2    50   Input ~ 0
+LCD_DB2
 Text HLabel 5900 3800 2    50   Input ~ 0
-LCD_DB6
-Text HLabel 5900 4300 2    50   Input ~ 0
-LCD_DB2
-Text HLabel 5900 3700 2    50   Input ~ 0
 LCD_DB7
 $Comp
@@
 	8900 3100 9200 3100
 Wire Wire Line
+	5600 3100 5900 3100
+Wire Wire Line
+	4000 4900 4300 4900
+Wire Wire Line
+	5600 4400 5900 4400
+Wire Wire Line
+	4000 5200 4300 5200
+Wire Wire Line
+	4300 5100 4000 5100
+Wire Wire Line
+	4000 5000 4300 5000
+Wire Wire Line
+	5600 4500 5900 4500
+Wire Wire Line
+	5900 3800 5600 3800
+Wire Wire Line
+	5600 3400 5900 3400
+Wire Wire Line
+	5900 3300 5600 3300
+Wire Wire Line
 	5600 3200 5900 3200
 Wire Wire Line
-	5900 3100 5600 3100
-Wire Wire Line
-	4300 5200 4000 5200
-Wire Wire Line
-	4000 5100 4300 5100
-Wire Wire Line
-	4300 5000 4000 5000
-Wire Wire Line
-	5900 3800 5600 3800
-Wire Wire Line
-	5600 4300 5900 4300
-Wire Wire Line
-	5900 3700 5600 3700
-Wire Wire Line
-	5600 3500 5900 3500
-Wire Wire Line
-	5900 3400 5600 3400
-Wire Wire Line
-	5600 3300 5900 3300
-Wire Wire Line
 	5900 5000 5600 5000
 Wire Wire Line
@@
 Wire Wire Line
 	8800 1800 9200 1800
+Text HLabel 5900 5500 2    50   Input ~ 0
+SW_1
 Text HLabel 4000 4600 0    50   Input ~ 0
-SW_1
+SW_2
 Text HLabel 4000 4700 0    50   Input ~ 0
-SW_2
+SW_3
 Text HLabel 4000 4800 0    50   Input ~ 0
-SW_3
-Text HLabel 4000 4900 0    50   Input ~ 0
 SW_4
 Text HLabel 3950 4100 0    50   Input ~ 0
@@
 POT_4
 Wire Wire Line
+	3950 4400 4300 4400
+Wire Wire Line
+	3950 4100 4300 4100
+Wire Wire Line
+	4300 4300 3950 4300
+Wire Wire Line
+	8800 1800 8800 5400
+Wire Wire Line
+	8900 3100 8900 5300
+Wire Wire Line
+	5900 5500 5600 5500
+Wire Wire Line
+	4300 4600 4000 4600
+Wire Wire Line
+	4000 4700 4300 4700
+Wire Wire Line
+	4300 4800 4000 4800
+Wire Wire Line
 	3950 4200 4300 4200
 Wire Wire Line
-	3950 4400 4300 4400
-Wire Wire Line
-	3950 4100 4300 4100
-Wire Wire Line
-	4300 4300 3950 4300
-Wire Wire Line
-	8800 1800 8800 5400
-Wire Wire Line
-	8900 3100 8900 5300
-Wire Wire Line
-	5600 3600 7350 3600
-Connection ~ 7350 3600
-Wire Wire Line
-	4000 4600 4300 4600
-Wire Wire Line
-	4300 4700 4000 4700
-Wire Wire Line
-	4000 4800 4300 4800
-Wire Wire Line
-	4300 4900 4000 4900
+	7350 3500 5600 3500
+Connection ~ 7350 3500
+Text HLabel 5900 3600 2    50   Input ~ 0
+SWDIO
+Wire Wire Line
+	5900 3600 5600 3600
+Text HLabel 5900 4300 2    50   Input ~ 0
+SWO
+Wire Wire Line
+	5900 4300 5600 4300
+Text HLabel 5900 3700 2    50   Input ~ 0
+SWCLK
+Wire Wire Line
+	5900 3700 5600 3700
 $EndSCHEMATC

Commit message: Add water pump output
Connections:
- net labels added: Water_Pump_PWM
- wire segments 159 -> 160
Changed lines of the file:
@@
 $Descr A4 11693 8268
 encoding utf-8
-Sheet 2 5
+Sheet 2 6
 Title ""
 Date ""
@@
 Wire Wire Line
 	5900 3700 5600 3700
+Text HLabel 5900 4600 2    50   Input ~ 0
+Water_Pump_PWM
+Wire Wire Line
+	5900 4600 5600 4600
 $EndSCHEMATC

Commit message: Add BOM
Parts:
- U301: Digikey (none) -> 497-17184-ND
Changed lines of the file:
@@
 F 2 "Package_QFP:LQFP-64_10x10mm_P0.5mm" H 4400 2200 50  0001 R CNN
 F 3 "http://www.st.com/st-web-ui/static/active/en/resource/technical/document/datasheet/DM00330506.pdf" H 5000 3900 50  0001 C CNN
+F 4 "497-17184-ND" H 5000 3900 50  0001 C CNN "Digikey"
 	1    5000 3900
 	1    0    0    -1

Commit message: Add PIN functions
Other:
- note added: "PB6 Water_Pump_PWM TIM4_CH1\nPC0 POT_1 ADC1_IN10\nPC1 POT_2 ADC1_IN11\nPC2 POT_3 ADC1_IN12\nPC3 POT_4 ADC1_IN13"
Changed lines of the file:
@@
 Wire Wire Line
 	5900 4600 5600 4600
+Text Notes 1100 5400 0    50   ~ 0
+PB6 Water_Pump_PWM TIM4_CH1\nPC0 POT_1 ADC1_IN10\nPC1 POT_2 ADC1_IN11\nPC2 POT_3 ADC1_IN12\nPC3 POT_4 ADC1_IN13
 $EndSCHEMATC

Commit message: Stepper pulse output description
Other:
- note added: "PB6 Water_Pump_PWM TIM4_CH1\nPB14 Stepper_PUL TIM12_CH1\nPC0 POT_1 ADC1_IN10\nPC1 POT_2 ADC1_IN11\nPC2 POT_3 ADC1_IN12\nPC3 POT_4 ADC1_IN13"
- note removed: "PB6 Water_Pump_PWM TIM4_CH1\nPC0 POT_1 ADC1_IN10\nPC1 POT_2 ADC1_IN11\nPC2 POT_3 ADC1_IN12\nPC3 POT_4 ADC1_IN13"
Changed lines of the file:
@@
 	5900 4600 5600 4600
 Text Notes 1100 5400 0    50   ~ 0
-PB6 Water_Pump_PWM TIM4_CH1\nPC0 POT_1 ADC1_IN10\nPC1 POT_2 ADC1_IN11\nPC2 POT_3 ADC1_IN12\nPC3 POT_4 ADC1_IN13
+PB6 Water_Pump_PWM TIM4_CH1\nPB14 Stepper_PUL TIM12_CH1\nPC0 POT_1 ADC1_IN10\nPC1 POT_2 ADC1_IN11\nPC2 POT_3 ADC1_IN12\nPC3 POT_4 ADC1_IN13
 $EndSCHEMATC
