File: hardware/edm_control_board/cad/controller.sch (KiCad schematic (older format))
At the start: 26 parts, among them Q201 BSS214NW, Q202 BSS214NW, Q203 BSS214NW, Q204 BSS214NW, U301 STM32F722RETx, Y201 25M

Commit message: Change C211, C212 from 0402 to 0805
Parts:
- C211, C212: Digikey 311-1442-1-ND -> 311-3425-1-ND
Changed lines of the file:
@@
 F 2 "Capacitor_SMD:C_0805_2012Metric" H 4038 2900 50  0001 C CNN
 F 3 "~" H 4000 3050 50  0001 C CNN
-F 4 "311-1442-1-ND" H 4000 3050 50  0001 C CNN "Digikey"
+F 4 "311-3425-1-ND" H 4000 3050 50  0001 C CNN "Digikey"
 	1    4000 3050
 	1    0    0    -1
@@
 F 2 "Capacitor_SMD:C_0805_2012Metric" H 3588 2900 50  0001 C CNN
 F 3 "~" H 3550 3050 50  0001 C CNN
-F 4 "311-1442-1-ND" H 3550 3050 50  0001 C CNN "Digikey"
+F 4 "311-3425-1-ND" H 3550 3050 50  0001 C CNN "Digikey"
 	1    3550 3050
 	1    0    0    -1

Commit message: Change C208, C210 from 0402 to 0805
Parts:
- C208, C210: Digikey 311-1641-1-ND -> 311-1100-1-ND
Changed lines of the file:
@@
 F 2 "Capacitor_SMD:C_0805_2012Metric" H 3188 4050 50  0001 C CNN
 F 3 "~" H 3150 4200 50  0001 C CNN
-F 4 "311-1641-1-ND" H 3150 4200 50  0001 C CNN "Digikey"
+F 4 "311-1100-1-ND" H 3150 4200 50  0001 C CNN "Digikey"
 	1    3150 4200
 	1    0    0    -1
@@
 F 2 "Capacitor_SMD:C_0805_2012Metric" H 2688 4050 50  0001 C CNN
 F 3 "~" H 2650 4200 50  0001 C CNN
-F 4 "311-1641-1-ND" H 2650 4200 50  0001 C CNN "Digikey"
+F 4 "311-1100-1-ND" H 2650 4200 50  0001 C CNN "Digikey"
 	1    2650 4200
 	1    0    0    -1

Commit message: Add NRST to SWD connector
Connections:
- net labels added: NRST
- wire segments 160 -> 163
Changed lines of the file:
@@
 	3100 2500 4300 2500
 Wire Wire Line
-	2700 2300 4300 2300
+	2700 2300 3000 2300
 Connection ~ 2700 2300
 Wire Wire Line
@@
 Text Notes 1100 5400 0    50   ~ 0
 PB6 Water_Pump_PWM TIM4_CH1\nPB14 Stepper_PUL TIM12_CH1\nPC0 POT_1 ADC1_IN10\nPC1 POT_2 ADC1_IN11\nPC2 POT_3 ADC1_IN12\nPC3 POT_4 ADC1_IN13
+Text HLabel 2900 2150 0    50   Input ~ 0
+NRST
+Wire Wire Line
+	2900 2150 3000 2150
+Wire Wire Line
+	3000 2150 3000 2300
+Connection ~ 3000 2300
+Wire Wire Line
+	3000 2300 4300 2300
 $EndSCHEMATC

Commit message: Update schematics with new STM32 symbol
Connections:
- wire segments 163 -> 151
