File: hardware/edm_control_board/cad/user_interface.sch (KiCad schematic (older format))
At the start: 9 parts, among them SW401 SW_Push, SW402 SW_Push, SW403 SW_Push, SW404 SW_Push, U401 NHD-0420H1Z

Commit message: Add SWD connector
Parts:
- renumbered RV401 to RV501, RV402 to RV502, RV403 to RV503, RV404 to RV504, SW401 to SW501, SW402 to SW502, SW403 to SW503, SW404 to SW504, U401 to U501
Changed lines of the file:
@@
 $EndDescr
 $Comp
-L Device:POT RV401
+L Device:POT RV501
 U 1 1 5A8932B6
 P 7400 2650
-F 0 "RV401" H 7330 2696 50  0000 R CNN
+F 0 "RV501" H 7330 2696 50  0000 R CNN
 F 1 "POT" H 7330 2605 50  0000 R CNN
 F 2 "Potentiometer_THT:Potentiometer_TT_P0915N" H 7400 2650 50  0001 C CNN
@@
 $EndComp
 $Comp
-L Device:POT RV403
+L Device:POT RV503
 U 1 1 5A893372
 P 7400 4350
-F 0 "RV403" H 7330 4396 50  0000 R CNN
+F 0 "RV503" H 7330 4396 50  0000 R CNN
 F 1 "POT" H 7330 4305 50  0000 R CNN
 F 2 "Potentiometer_THT:Potentiometer_TT_P0915N" H 7400 4350 50  0001 C CNN
@@
 $EndComp
 $Comp
-L Device:POT RV402
+L Device:POT RV502
 U 1 1 5A893438
 P 9200 2650
-F 0 "RV402" H 9130 2696 50  0000 R CNN
+F 0 "RV502" H 9130 2696 50  0000 R CNN
 F 1 "POT" H 9130 2605 50  0000 R CNN
 F 2 "Potentiometer_THT:Potentiometer_TT_P0915N" H 9200 2650 50  0001 C CNN
@@
 $EndComp
 $Comp
-L Device:POT RV404
+L Device:POT RV504
 U 1 1 5A89343E
 P 9200 4350
-F 0 "RV404" H 9130 4396 50  0000 R CNN
+F 0 "RV504" H 9130 4396 50  0000 R CNN
 F 1 "POT" H 9130 4305 50  0000 R CNN
 F 2 "Potentiometer_THT:Potentiometer_TT_P0915N" H 9200 4350 50  0001 C CNN
@@
 $EndComp
 $Comp
-L Switch:SW_Push SW401
+L Switch:SW_Push SW501
 U 1 1 5A893485
 P 2750 4850
-F 0 "SW401" H 2750 5135 50  0000 C CNN
+F 0 "SW501" H 2750 5135 50  0000 C CNN
 F 1 "SW_Push" H 2750 5044 50  0000 C CNN
 F 2 "Button_Switch_THT:SW_PUSH_CK_PVA1" H 2750 5050 50  0001 C CNN
@@
 $EndComp
 $Comp
-L Switch:SW_Push SW403
+L Switch:SW_Push SW503
 U 1 1 5A893559
 P 2750 6050
-F 0 "SW403" H 2750 6335 50  0000 C CNN
+F 0 "SW503" H 2750 6335 50  0000 C CNN
 F 1 "SW_Push" H 2750 6244 50  0000 C CNN
 F 2 "Button_Switch_THT:SW_PUSH_CK_PVA1" H 2750 6250 50  0001 C CNN
@@
 $EndComp
 $Comp
-L Switch:SW_Push SW402
+L Switch:SW_Push SW502
 U 1 1 5A8935E5
 P 4350 4850
-F 0 "SW402" H 4350 5135 50  0000 C CNN
+F 0 "SW502" H 4350 5135 50  0000 C CNN
 F 1 "SW_Push" H 4350 5044 50  0000 C CNN
 F 2 "Button_Switch_THT:SW_PUSH_CK_PVA1" H 4350 5050 50  0001 C CNN
@@
 $EndComp
 $Comp
-L Switch:SW_Push SW404
+L Switch:SW_Push SW504
 U 1 1 5A8935EB
 P 4350 6050
-F 0 "SW404" H 4350 6335 50  0000 C CNN
+F 0 "SW504" H 4350 6335 50  0000 C CNN
 F 1 "SW_Push" H 4350 6244 50  0000 C CNN
 F 2 "Button_Switch_THT:SW_PUSH_CK_PVA1" H 4350 6250 50  0001 C CNN
@@
 $EndComp
 $Comp
-L Display_Character:NHD-0420H1Z U401
+L Display_Character:NHD-0420H1Z U501
 U 1 1 5A87AF27
 P 4050 2650
-F 0 "U401" H 4150 3400 50  0000 L CNN
+F 0 "U501" H 4150 3400 50  0000 L CNN
 F 1 "NHD-0420H1Z" H 4150 3300 50  0000 L CNN
 F 2 "Display:NHD-0420H1Z" H 4150 1850 50  0001 C CNN

Commit message: Old
Parts:
- RV501, RV502, RV503, RV504: Digikey (none) -> 987-1278-ND
- SW501, SW502, SW503, SW504: Digikey (none) -> 401-1137-ND
- U501: Digikey (none) -> NHD-0420H1Z-FSW-GBW-33V3-ND
Changed lines of the file:
@@
 F 2 "Potentiometer_THT:Potentiometer_TT_P0915N" H 7400 2650 50  0001 C CNN
 F 3 "~" H 7400 2650 50  0001 C CNN
+F 4 "987-1278-ND" H 7400 2650 50  0001 C CNN "Digikey"
 	1    7400 2650
 	-1   0    0    -1
@@
 F 2 "Potentiometer_THT:Potentiometer_TT_P0915N" H 7400 4350 50  0001 C CNN
 F 3 "~" H 7400 4350 50  0001 C CNN
+F 4 "987-1278-ND" H 7400 4350 50  0001 C CNN "Digikey"
 	1    7400 4350
 	-1   0    0    -1
@@
 F 2 "Potentiometer_THT:Potentiometer_TT_P0915N" H 9200 2650 50  0001 C CNN
 F 3 "~" H 9200 2650 50  0001 C CNN
+F 4 "987-1278-ND" H 9200 2650 50  0001 C CNN "Digikey"
 	1    9200 2650
 	-1   0    0    -1
@@
 F 2 "Potentiometer_THT:Potentiometer_TT_P0915N" H 9200 4350 50  0001 C CNN
 F 3 "~" H 9200 4350 50  0001 C CNN
+F 4 "987-1278-ND" H 9200 4350 50  0001 C CNN "Digikey"
 	1    9200 4350
 	-1   0    0    -1
@@
 F 2 "Button_Switch_THT:SW_PUSH_CK_PVA1" H 2750 5050 50  0001 C CNN
 F 3 "" H 2750 5050 50  0001 C CNN
+F 4 "401-1137-ND" H 2750 4850 50  0001 C CNN "Digikey"
 	1    2750 4850
 	1    0    0    -1
@@
 F 2 "Button_Switch_THT:SW_PUSH_CK_PVA1" H 2750 6250 50  0001 C CNN
 F 3 "" H 2750 6250 50  0001 C CNN
+F 4 "401-1137-ND" H 2750 6050 50  0001 C CNN "Digikey"
 	1    2750 6050
 	1    0    0    -1
@@
 F 2 "Button_Switch_THT:SW_PUSH_CK_PVA1" H 4350 5050 50  0001 C CNN
 F 3 "" H 4350 5050 50  0001 C CNN
+F 4 "401-1137-ND" H 4350 4850 50  0001 C CNN "Digikey"
 	1    4350 4850
 	1    0    0    -1
@@
 F 2 "Button_Switch_THT:SW_PUSH_CK_PVA1" H 4350 6250 50  0001 C CNN
 F 3 "" H 4350 6250 50  0001 C CNN
+F 4 "401-1137-ND" H 4350 6050 50  0001 C CNN "Digikey"
 	1    4350 6050
 	1    0    0    -1
@@
 F 2 "Display:NHD-0420H1Z" H 4150 1850 50  0001 C CNN
 F 3 "http://www.newhavendisplay.com/specs/NHD-0420H1Z-FSW-GBW-33V3.pdf" H 4150 2550 50  0001 C CNN
+F 4 "NHD-0420H1Z-FSW-GBW-33V3-ND" H 4050 2650 50  0001 C CNN "Digikey"
 	1    4050 2650
 	1    0    0    -1
@@
 	1    0    0    -1
 $EndComp
-Wire Wire Line
-	4050 3450 4050 3350
 Text HLabel 7100 2650 0    50   Input ~ 0
 POT_1
@@
 Wire Wire Line
 	9200 4200 9200 4100
+Wire Wire Line
+	4050 3350 4050 3450
 $EndSCHEMATC
